File: meshtastic.kicad_sch (KiCad schematic)
At the start: 52 parts, among them J1 I2C1, J2 SPI BUS, J6 Conn_01x02, J7 I2C2, Q1 AO3401A, Q3 CSD16301Q2, Q4 CSD16301Q2, U1 XIAO-ESP32-C6-SMD, U4 BQ297xy, U6 TPS2116DRL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

Commit message: commits for assembly
Parts:
- Q3, Q4: LCSC Part (none) -> C140340
- U4: value BQ297xy -> BQ29700; LCSC Part (none) -> C183096
Changed lines of the file:
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@@
 		)
 	)
+	(text_box "todo: add VBUS inrush current limiting\r\nThe TPS2116 has this, but only for inital power on, not switching from Battery to VBUS"
+		(exclude_from_sim no)
+		(at 121.92 66.04 0)
+		(size 39.37 12.7)
+		(margins 0.9525 0.9525 0.9525 0.9525)
+		(stroke
+			(width 0)
+			(type solid)
+		)
+		(fill
+			(type none)
+		)
+		(effects
+			(font
+				(size 1.27 1.27)
+			)
+			(justify left top)
+		)
+	)
 	(junction
 		(at 152.4 58.42)
@@
 			)
 		)
+		(property "LCSC Part" "C140340"
+			(at 124.46 176.53 0)
+			(hide yes)
+			(show_name no)
+			(do_not_autoplace no)
+			(effects
+				(font
+					(size 1.27 1.27)
+				)
+			)
+		)
+		(property "Voltage Rating" ""
+			(at 124.46 176.53 0)
+			(hide yes)
+			(show_name no)
+			(do_not_autoplace no)
+			(effects
+				(font
+					(size 1.27 1.27)
+				)
+			)
+		)
+		(property "Tolerance" ""
+			(at 124.46 176.53 0)
+			(hide yes)
+			(show_name no)
+			(do_not_autoplace no)
+			(effects
+				(font
+					(size 1.27 1.27)
+				)
+			)
+		)
 		(pin "4"
 		)
@@
 			)
 		)
+		(property "LCSC Part" "C140340"
+			(at 114.3 171.45 0)
+			(hide yes)
+			(show_name no)
+			(do_not_autoplace no)
+			(effects
+				(font
+					(size 1.27 1.27)
+				)
+			)
+		)
+		(property "Voltage Rating" ""
+			(at 114.3 171.45 0)
+			(hide yes)
+			(show_name no)
+			(do_not_autoplace no)
+			(effects
+				(font
+					(size 1.27 1.27)
+				)
+			)
+		)
+		(property "Tolerance" ""
+			(at 114.3 171.45 0)
+			(hide yes)
+			(show_name no)
+			(do_not_autoplace no)
+			(effects
+				(font
+					(size 1.27 1.27)
+				)
+			)
+		)
 		(pin "4"
 		)
@@
 			)
 		)
-		(property "Value" "BQ297xy"
+		(property "Value" "BQ29700"
 			(at 114.3 143.51 0)
 			(show_name no)
@@
 			(at 114.3 151.13 0)
 			(hide yes)
+			(show_name no)
+			(do_not_autoplace no)
+			(effects
+				(font
+					(size 1.27 1.27)
+				)
+			)
+		)
+		(property "LCSC Part" "C183096"
+			(at 114.3 151.13 0)
+			(hide yes)
+			(show_name no)
+			(do_not_autoplace no)
+			(effects
+				(font
+					(size 1.27 1.27)
+				)
+			)
+		)
+		(property "Voltage Rating" ""
+			(at 114.3 151.13 0)
+			(hide yes)
+			(show_name no)
+			(do_not_autoplace no)
+			(effects
+				(font
+					(size 1.27 1.27)
+				)
+			)
+		)
+		(property "Tolerance" ""
+			(at 114.3 151.13 0)
+			(hide yes)
