File: meshtastic.kicad_sch (KiCad schematic)
At the start: 52 parts, among them J1 I2C1, J2 SPI BUS, J6 Conn_01x02, J7 I2C2, Q1 AO3401A, Q3 CSD16301Q2, Q4 CSD16301Q2, U1 XIAO-ESP32-C6-SMD, U4 BQ29700, U6 TPS2116DRL, U7 TPS61033DRLR

Commit message: Update schematics and rework NEO-M9N reader sketches
Co-Authored-By: Claude Opus 4.8 <noreply@anthropic.com>
Parts:
- removed R7: 10k, Resistor_SMD:R_0402_1005Metric, symbol Device:R_Small
Other:
- sheet GNSS ports: added none; removed RESET
