File: meshtastic.kicad_sch (KiCad schematic)
At the start: 51 parts, among them J1 I2C1, J2 SPI BUS, J6 Conn_01x02, J7 I2C2, Q1 AO3401A, Q3 CSD16301Q2, Q4 CSD16301Q2, U1 XIAO-ESP32-C6-SMD, U4 BQ29700, U6 TPS2116DRL, U7 TPS61033DRLR

Commit message: pcb updates
Parts:
- BT1: value Battery_Cell -> 18650 Lithium-Ion
- J6: LCSC C2905009 -> (none); LCSC Part (none) -> C2905009
Other:
- note added: "todo: switch to 21700"

Commit message: next revision pcb progress
Parts:
- removed BT1: 18650 Lithium-Ion, Battery:BatteryHolder_Keystone_1042_1x18650, symbol Device:Battery_Cell
- removed C19, C21: 100nF, Capacitor_SMD:C_0402_1005Metric, symbol Device:C_Small
- removed C20, C22, C23, C24: 10uF, Capacitor_SMD:C_0402_1005Metric, symbol Device:C_Small
- removed FB1: FerriteBead, Inductor_SMD:L_0603_1608Metric, symbol Device:FerriteBead
- removed J6: Conn_01x02, Connector_Molex:Molex_PicoBlade_53261-0271_1x02-1MP_P1.25mm_Horizontal, symbol Connector_Generic_MountingPin:Conn_01x02_MountingPin
- removed L2: 470nH, Inductor_SMD:L_1008_2520Metric_Pad1.43x2.20mm_HandSolder, symbol Device:L
- removed Q1: AO3401A, Package_TO_SOT_SMD:SOT-23, symbol Transistor_FET:AO3401A
- removed Q3, Q4: CSD16301Q2, Package_SON:Texas_DQK, symbol Transistor_FET:CSD16301Q2
- removed R18: 10k, Resistor_SMD:R_0402_1005Metric, symbol Device:R_Small
- removed R19: 2.2k, Resistor_SMD:R_0402_1005Metric, symbol Device:R
- removed R20: 330, Resistor_SMD:R_0402_1005Metric, symbol Device:R_Small
- removed R22: 1k, Resistor_SMD:R_0402_1005Metric, symbol Device:R_Small
- removed R23: 2M, Resistor_SMD:R_0402_1005Metric, symbol Device:R_Small
- removed R24: 680k, Resistor_SMD:R_0402_1005Metric, symbol Device:R_Small
- removed U4: BQ29700, Package_SON:WSON-6_1.5x1.5mm_P0.5mm, symbol Battery_Management:BQ297xy
- removed U6: TPS2116DRL, Package_TO_SOT_SMD:SOT-583-8, symbol Power_Management:TPS2116DRL
- removed U7: TPS61033DRLR, Package_TO_SOT_SMD:SOT-583-8, symbol easyeda2kicad:TPS61033DRLR
- added F2, F3, F4: Littelfuse 0805L050WR, Fuse:Fuse_0805_2012Metric, symbol Device:Polyfuse_Small
- D4: value ESDS314DBVR-TP -> TI ESDS314DBVR; LCSC Part C5310975 -> C1847859; MPN ESDS314DBVR-TP -> ESDS314DBVR; Manufacturer TECH PUBLIC(台舟) -> (none)
- D5: value ESDS314DBVR-TP -> TI ESDS314DBVR; LCSC Part C5310975 -> C1847859; MPN ESDS314DBVR-TP -> ESDS314DBVR; Manufacturer TECH PUBLIC(台舟) -> ti
Connections:
- net +3V3: now also F2.1, F3.1, F4.1; no longer J1.1 (Pin_1), J2.1 (Pin_1), J7.1 (Pin_1)
- new net: F4.2, J7.1 (Pin_1)
- new net: F2.2, J2.1 (Pin_1)
- new net: F3.2, J1.1 (Pin_1)
- no-connect marks 7 -> 5
Other:
- added sheet Power_Management (Power.kicad_sch)
- note removed: "5V Switching Regulator"
- note removed: "BMS"
- note removed: "Power Muxer"
- note removed: "Reverse Polarity Protection"
- note removed: "todo: switch to 21700"
- moved on the sheet: H1, H2, H3, H4

Commit message: changes
Parts:
- removed C1, C2, C3, C5, C6, C7: 10uF, Capacitor_SMD:C_0402_1005Metric, symbol Device:C_Small
- removed C25, C4: 100nF, Capacitor_SMD:C_0402_1005Metric, symbol Device:C_Small
- removed R1, R2: 4.7k, Resistor_SMD:R_0402_1005Metric, symbol Device:R_Small
- removed R25, R26: 100k, Resistor_SMD:R_0402_1005Metric, symbol Device:R_Small
- removed R3, R4, R5, R6: 22, Resistor_SMD:R_0402_1005Metric, symbol Device:R_Small
- removed U1: XIAO-ESP32-C6-SMD, footprints:XIAO-ESP32-C6-SMD, symbol Seeed_Studio_XIAO_Series:XIAO-ESP32-C6-SMD
- added J8: GCT USB4105-GF-A-120, Connector_USB:USB_C_Receptacle_GCT_USB4105-xx-A_16P_TopMnt_Horizontal, symbol Connector:USB_C_Receptacle_USB2.0_16P
- added U7: ESP32-S3-WROOM-1, RF_Module:ESP32-S3-WROOM-1, symbol RF_Module:ESP32-S3-WROOM-1
Connections:
- new net: U7.1 (GND), U7.40 (GND), U7.41 (GND)
- new net: J8.A1 (GND), J8.A12 (GND), J8.B1 (GND), J8.B12 (GND)
- new net: J8.A4 (VBUS), J8.A9 (VBUS), J8.B4 (VBUS), J8.B9 (VBUS)
- no-connect marks 5 -> 1
