File: GNSS-NEO.kicad_sch (KiCad schematic)
At the start: 25 parts, among them J3 Conn_Coaxial, J4 Conn_Coaxial_Small, SW1 SW_Push, U2 NEO-M9N

Commit message: show to ppl
Parts:
- C10: value 100nF 16V -> 100nF; Voltage Rating (none) -> 16V
- R27, R28: footprint Resistor_SMD:R_0603_1608Metric -> Resistor_SMD:R_0402_1005Metric
Changed lines of the file:
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@@
 			)
 		)
-		(property "Footprint" "Resistor_SMD:R_0603_1608Metric"
+		(property "Footprint" "Resistor_SMD:R_0402_1005Metric"
 			(at 100.33 162.56 0)
 			(hide yes)
@@
 			)
 		)
-		(property "Footprint" "Resistor_SMD:R_0603_1608Metric"
+		(property "Footprint" "Resistor_SMD:R_0402_1005Metric"
 			(at 88.9 162.56 0)
 			(hide yes)
@@
 			)
 		)
-		(property "Value" "100nF 16V"
+		(property "Value" "100nF"
 			(at 84.328 179.07 90)
 			(show_name no)
@@
 			)
 		)
-		(property "Voltage Rating" ""
+		(property "Voltage Rating" "16V"
 			(at 83.82 176.53 0)
 			(hide yes)
