File: GNSS-NEO.kicad_sch (KiCad schematic)
At the start: 72 parts, among them J3 Conn_Coaxial, J4 Conn_Coaxial_Small, Q2 AO3401A, Q5 BSS138, SW1 SW_Push, SW2 SW_Push, U2 NEO-M9N, U8 TPS259474LRPWR

Commit message: changes
Parts:
- added C108, C93: 2.2uF, symbol Device:C_Small
- added D17: D_Schottky, symbol Device:D_Schottky
- added U11: TPS7A2033PDBVR, easyeda2kicad:SOT-23-5_L2.9-W1.6-P0.95-LS2.8-BR, symbol easyeda2kicad:TPS7A2033PDBVR
Connections:
- net +3V3: no longer C40.1, C41.2, C43.2, D13.1 (A1), R29.1, R41.1, U8.5 (IN)
- net +5V: now also C93.1, U11.1 (IN), U11.3 (EN)
- net GND: now also C108.2, C93.2, U11.2 (GND)
- net VCC_RF: now also D17.2 (A); no longer JP4.3 (B)
- new net: C108.1, C40.1, C41.2, C43.2, D13.1 (A1), R29.1, R41.1, U11.5 (OUT), U8.5 (IN)
- new net: D17.1 (K), JP4.3 (B)
- no-connect marks 2 -> 3
Other:
- note added: "High PSRR & Low Noise LDO"
- moved on the sheet: C16, C17, C40, C41, C43, C44, C45, D13, JP7, R29, R38, R40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
