File: LORA-E22.kicad_sch (KiCad schematic)
At the start: 16 parts, among them J5 Conn_Coaxial, U3 E22P-915M30S

Commit message: commits for assembly
Parts:
- D6: value SMAJ5.0A -> SMAJ3.3A
- D8: value BESDU0603 -> BESDU0603-14
Changed lines of the file:
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@@
 			)
 		)
-		(property "Value" "BESDU0603"
-			(at 121.158 109.22 90)
+		(property "Value" "BESDU0603-14"
+			(at 117.094 108.966 90)
 			(show_name no)
 			(do_not_autoplace no)
@@
 			)
 		)
-		(property "Value" "SMAJ5.0A"
+		(property "Value" "SMAJ3.3A"
 			(at 127 73.66 0)
 			(show_name no)

Commit message: show to ppl
Parts:
- C14, C18: Voltage Rating (none) -> 10V
Changed lines of the file:
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@@
 			)
 		)
-		(property "Voltage Rating" ""
+		(property "Voltage Rating" "10V"
 			(at 203.2 77.47 0)
 			(hide yes)
@@
 			)
 		)
-		(property "Voltage Rating" ""
+		(property "Voltage Rating" "10V"
 			(at 193.04 77.47 0)
 			(hide yes)
