File: battery.kicad_sch (KiCad schematic)
At the start: 86 parts, among them J6 Conn_01x02, Q5 AON7534, Q6 AON7534, Q7 TI CSD18512Q5B, SW3 RESET, U6 MAX17320G22+, U7 BQ25798

Commit message: journal update!
Parts:
- removed C63: 1nF, Capacitor_SMD:C_0402_1005Metric, symbol Device:C_Small
- removed C69: 100nF, Capacitor_SMD:C_0402_1005Metric, symbol Device:C_Small
- removed D3: SMF10A, Diode_SMD:D_SOD-123, symbol Device:D_TVS
- added C163, C164, C165: 10uF, Capacitor_SMD:C_1210_3225Metric, symbol Device:C_Small
- added D21: SMF10A, Diode_SMD:D_SOD-123, symbol Diode:SMF10A
- added JP6: ZVC, Jumper:SolderJumper-2_P1.3mm_Open_RoundedPad1.0x1.5mm, symbol Jumper:SolderJumper_2_Open
- added Q12: CSD18512Q5B, Package_SON:VSONP-8-1EP_5x6_P1.27mm, symbol Transistor_FET:CSD18532Q5B
- added Q13: CSD17581Q3A, Package_SON:VSON-8_3.3x3.3mm_P0.65mm_NexFET, symbol Transistor_FET:CSD17581Q3A
- added R120: 294, symbol Device:R_Small
- added R122: 100, Resistor_SMD:R_0402_1005Metric, symbol Device:R_Small
- C55, C56, C67, C76: Capacitor Rating (none) -> X7R; LCSC Part C6119785 -> C5142567
- C65: Voltage Rating 16V -> 25V
- Q7: value TI CSD18512Q5B -> CSD18512Q5B
- R31: now fitted
- R38: value 47k -> 24.3k
- R39: value 51.1k -> 68.1k
- SW3: value RESET -> POWER/RESET
Connections:
- net +PACK: now also Q13.5 (D); no longer U7.22 (BAT), U7.23 (BAT)
- net -BATT: now also D21.2 (A2)
- net GND: now also C74.2, C163.1, C164.2, C165.2; no longer C74.1
- net VSYS: now also C74.1, C163.2; no longer C74.2
- net at BT1.1 (+), C37.1, C38.1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: now also D21.1 (A1)
- net at C56.1, C57.1, C58.1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: now also Q12.5 (D); no longer Q7.1 (S), Q7.2 (S), Q7.3 (S)
- net at R31.1: now also JP6.2 (B); no longer U6.5 (ZVC)
- net at U7.24 (SDRV): now also Q13.4 (G)
- net at SW3.2: now also R122.1; no longer U7.12 (~{QON})
- net at R41.2, U7.11 (ACDRV1): now also R120.2
- new net: Q12.4 (G), R120.1
- new net: JP6.1 (A), U6.5 (ZVC)
- new net: C164.1, C165.1, Q13.1 (S), Q13.2 (S), Q13.3 (S), U7.22 (BAT), U7.23 (BAT)
- new net: Q12.1 (S), Q12.2 (S), Q12.3 (S), Q7.1 (S), Q7.2 (S), Q7.3 (S)
- new net: R122.2, U7.12 (~{QON})
Other:
- moved on the sheet: C40, C54, C55, C56, C57, C58, C59, C61, C62, C65, C67, C71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

Commit message: pcb layout!
Parts:
- removed C56: 100nF, Capacitor_SMD:C_0402_1005Metric, symbol Device:C_Small
- removed C57, C58, C59: 10uF, Capacitor_SMD:C_1210_3225Metric, symbol Device:C_Small
- removed Q12, Q7: CSD18512Q5B, Package_SON:VSONP-8-1EP_5x6_P1.27mm, symbol Transistor_FET:CSD18532Q5B
- added C71, C73, C74, C90: 10uF, Capacitor_SMD:C_1206_3216Metric, symbol Device:C_Small
- added C72, C91: 100nF, Capacitor_SMD:C_0402_1005Metric, symbol Device:C_Small
- added C79: 2.2uF, Capacitor_SMD:C_0805_2012Metric, symbol Device:C_Small
- added D7: SMF24A, Diode_SMD:D_SOD-123F, symbol Diode:SMF24A
- added D9: SS36B, Diode_SMD:D_SMB, symbol Device:D_Schottky
- added J10: SOLAR, Connector_JST:JST_PH_S2B-PH-SM4-TB_1x02-1MP_P2.00mm_Horizontal, symbol Connector:Conn_01x02_Socket
- added Q10, Q9: SI2308, Package_TO_SOT_SMD:SOT-23, symbol Transistor_FET:Q_NMOS_GSD
- added Q7, Q8: CSD18512Q5B, Package_SON:VSONP-8-1EP_5x6_P1.27mm, symbol Transistor_FET:Q_NMOS_DGS
- added R60, R61: 294, Resistor_SMD:R_0402_1005Metric, symbol Device:R_Small
- added R62: 2, Resistor_SMD:R_0402_1005Metric, symbol Device:R_Small
- added TH2, TH3: 103AT 10k, Resistor_SMD:R_0603_1608Metric, symbol Device:Thermistor_NTC
- BT1, BT2: footprint easyeda2kicad:BAT-TH_BH-21700-A5BJ001 -> easyeda2kicad:BAT-SMD_L82.5.5-W25-BH-21700-B1BJ001; LCSC Part (none) -> C20606791
- C47: renamed from C37; footprint (none) -> Capacitor_SMD:C_0402_1005Metric; LCSC Part (none) -> C7472948
- C48: renamed from C38; value 22uF -> 10uF; LCSC Part (none) -> C6119892
- C49: renamed from C39; footprint (none) -> Capacitor_SMD:C_0402_1005Metric; Capacitor Rating (none) -> X7R; LCSC Part (none) -> C5272680
- C50: renamed from C40; footprint (none) -> Capacitor_SMD:C_0402_1005Metric; Capacitor Rating (none) -> X7R; LCSC Part (none) -> C5272680
- C51: renamed from C41; footprint (none) -> Capacitor_SMD:C_0402_1005Metric; Capacitor Rating (none) -> X7R; LCSC Part (none) -> C5272680
- C52: renamed from C42; footprint (none) -> Capacitor_SMD:C_0402_1005Metric; LCSC Part (none) -> C7472948
- C53: renamed from C43; footprint (none) -> Capacitor_SMD:C_0402_1005Metric; LCSC Part (none) -> C49333230
- C54: renamed from C44; footprint (none) -> Capacitor_SMD:C_0402_1005Metric; Capacitor Rating (none) -> X7R; LCSC Part (none) -> C5272680
- C55: renamed from C45; LCSC Part (none) -> C49333230
- C56: renamed from C46; LCSC Part (none) -> C49333230
- C57: renamed from C64; footprint Capacitor_SMD:C_1210_3225Metric -> Capacitor_SMD:C_1206_3216Metric; LCSC Part C7472976 -> C49326770
- C58: renamed from C47; LCSC Part (none) -> C49333230
- C59: renamed from C66; footprint Capacitor_SMD:C_1210_3225Metric -> Capacitor_SMD:C_1206_3216Metric; LCSC Part C7472976 -> C49326770
- C60: renamed from C68; footprint Capacitor_SMD:C_1210_3225Metric -> Capacitor_SMD:C_1206_3216Metric; LCSC Part C7472976 -> C49326770
- C61: renamed from C48; footprint (none) -> Capacitor_SMD:C_0402_1005Metric; Capacitor Rating (none) -> X7R; LCSC Part (none) -> C5272680
- C62: renamed from C54; LCSC Part (none) -> C17702473
- C63: renamed from C70; footprint Capacitor_SMD:C_1210_3225Metric -> Capacitor_SMD:C_1206_3216Metric; LCSC Part C7472976 -> C49326770
- C64: renamed from C55; LCSC Part C5142567 -> C5272680
- C65: renamed from C163; footprint Capacitor_SMD:C_1210_3225Metric -> Capacitor_SMD:C_1206_3216Metric; LCSC Part C7472976 -> C49326770
- C66: renamed from C49; footprint (none) -> Capacitor_SMD:C_0402_1005Metric; Capacitor Rating (none) -> X7R; LCSC Part (none) -> C5272680
- C67: renamed from C50; LCSC Part C33546010 -> C6119892
- C68: renamed from C51; LCSC Part C33546010 -> C6119892
- C69: renamed from C52; LCSC Part C33546010 -> C6119892
- C70: renamed from C53; LCSC Part C33546010 -> C6119892
- C75: renamed from C61; LCSC Part (none) -> C5142571
- C76: renamed from C62; LCSC Part (none) -> C5142571
- C77: renamed from C60; LCSC Part (none) -> C5142571
- C78: renamed from C65; LCSC Part (none) -> C22367829
- C80: renamed from C67; LCSC Part C5142567 -> C5272680
- C82: renamed from C71; footprint Capacitor_SMD:C_1210_3225Metric -> Capacitor_SMD:C_1206_3216Metric; LCSC Part C7472976 -> C49326770
- C84: renamed from C165; footprint Capacitor_SMD:C_1210_3225Metric -> Capacitor_SMD:C_1206_3216Metric; LCSC Part C7472976 -> C49326770
- C85: renamed from C164; footprint Capacitor_SMD:C_1210_3225Metric -> Capacitor_SMD:C_1206_3216Metric; LCSC Part C7472976 -> C49326770
- C86: renamed from C75; footprint Capacitor_SMD:C_1210_3225Metric -> Capacitor_SMD:C_1206_3216Metric; LCSC Part C7472976 -> C49326770
- C87: renamed from C77; footprint Capacitor_SMD:C_1210_3225Metric -> Capacitor_SMD:C_1206_3216Metric; LCSC Part C7472976 -> C49326770
- C88: renamed from C78; footprint Capacitor_SMD:C_1210_3225Metric -> Capacitor_SMD:C_1206_3216Metric; LCSC Part C7472976 -> C49326770
- C89: renamed from C76; LCSC Part C5142567 -> C5272680
- C92: renamed from C74; footprint Capacitor_SMD:C_1210_3225Metric -> Capacitor_SMD:C_1206_3216Metric; LCSC Part C7472976 -> C49326770
- D8: renamed from D5; footprint (none) -> LED_SMD:LED_0805_2012Metric; LCSC Part (none) -> C19171393
- F5: renamed from F4; footprint (none) -> Fuse:Fuse_2920_7451Metric; LCSC Part (none) -> C50338483
- J9: renamed from J6; now not fitted
- Q11: renamed from Q13; LCSC Part (none) -> C2861705
- R39: renamed from R24; LCSC Part (none) -> C319867
- R40: renamed from R25; LCSC Part (none) -> C319867
- R41: renamed from R26; footprint (none) -> Resistor_SMD:R_0805_2012Metric_Pad1.20x1.40mm_HandSolder; LCSC Part (none) -> C42454064
- R42: renamed from R27; footprint (none) -> Resistor_SMD:R_0402_1005Metric; LCSC Part (none) -> C1883546
- R43: renamed from R28; footprint (none) -> Resistor_SMD:R_0402_1005Metric; LCSC Part (none) -> C48533754
- R44: renamed from R29; footprint (none) -> Resistor_SMD:R_0402_1005Metric; LCSC Part (none) -> C55174701
- R45: renamed from R30; footprint (none) -> Resistor_SMD:R_0402_1005Metric; LCSC Part (none) -> C48533754
- R46: renamed from R32; footprint (none) -> Resistor_SMD:R_0402_1005Metric; LCSC Part (none) -> C2902636
- R47: renamed from R31; value 330 0.75w -> 330; footprint Resistor_SMD:R_2010_5025Metric -> Resistor_SMD:R_1210_3225Metric; LCSC Part (none) -> C51048356; Power Rating (none) -> 750mW
- R48: renamed from R33; footprint (none) -> Resistor_SMD:R_0402_1005Metric; LCSC Part (none) -> C55174701
- R49: renamed from R35; LCSC Part (none) -> C881429
- R50: renamed from R34; footprint (none) -> Resistor_SMD:R_0402_1005Metric; LCSC Part (none) -> C2902636
- R51: renamed from R36; LCSC Part (none) -> C861485
- R52: renamed from R37; LCSC Part (none) -> C2989442
- R53: renamed from R41; footprint (none) -> Resistor_SMD:R_0402_1005Metric; LCSC Part (none) -> C852689
- R54: renamed from R38; LCSC Part (none) -> C2681615
- R55: renamed from R39; LCSC Part (none) -> C5355251
- R56: renamed from R40; LCSC Part (none) -> C2984406
- R57: renamed from R120; footprint (none) -> Resistor_SMD:R_0402_1005Metric; LCSC Part (none) -> C852689
- R58: renamed from R42; LCSC Part (none) -> C24265089
- R59: renamed from R122; LCSC Part (none) -> C55174701
- R63: renamed from R43; LCSC Part (none) -> C55174701
- R64: renamed from R45; LCSC Part (none) -> C54530782
- R65: renamed from R44; LCSC Part (none) -> C54530782
- R66: renamed from R46; LCSC Part (none) -> C29269950
- SW3: footprint (none) -> Button_Switch_SMD:SW_Push_SPST_NO_Alps_SKRK; LCSC Part (none) -> C2681476
- TH1: footprint (none) -> Resistor_SMD:R_0603_1608Metric; LCSC Part (none) -> C3154661
- TH4: renamed from TH2; footprint (none) -> Resistor_SMD:R_0603_1608Metric; LCSC Part (none) -> C3154661
- TH5: renamed from TH3; footprint (none) -> Resistor_SMD:R_0603_1608Metric; LCSC Part (none) -> C3154661
- TP3: footprint (none) -> TestPoint:TestPoint_Pad_D1.5mm
- TP4: footprint (none) -> TestPoint:TestPoint_2Pads_Pitch2.54mm_Drill0.8mm
- U8: renamed from U7; LCSC Part (none) -> C2876593
- renumbered C73 to C81, C72 to C83, D21 to D5, D4 to D6, JP6 to JP7, U6 to U7
Connections:
- net -BATT: now also TH2.2, TH3.2
- net GND: now also C71.1, C72.1, C73.1, C74.1, C79.2, C90.1, C91.2, D7.2 (A2), D9.2 (A), J10.2 (Pin_2); no longer U8.10 (ACDRV2)
- net PPHV: now also Q7.1 (D)
- net at R57.1: now also Q8.2 (G)
- net at U8.2 (VBUS), U8.3 (VBUS): now also C71.2, C72.2, C73.2, C74.2, Q8.1 (D), Q9.3 (D); no longer U8.8 (VAC2)
- net at U7.18 (TH3): now also TH3.1
- net at U7.19 (TH4): now also TH2.1
- net at R53.1: now also Q7.2 (G)
- new net: Q10.1 (G), R61.1
- new net: Q10.2 (S), Q9.2 (S)
- new net: R60.2, R61.2, U8.10 (ACDRV2)
- new net: Q9.1 (G), R60.1
- new net: Q7.3 (S), Q8.3 (S)
- new net: C79.1, R62.2
- new net SOLAR: C90.2, C91.1, D7.1 (A1), D9.1 (K), J10.1 (Pin_1), Q10.3 (D), R62.1, U8.8 (VAC2)
- no-connect marks 5 -> 3
Other:
- note added: "4 x 10uF 1206"
- note removed: "4 x 10uF 1210"

Commit message: organize repo and schematic
Parts:
- J9: value Conn_01x02 -> BAT_PORT
Other:
- moved on the sheet: BT1, BT2, C47, C48, C49, C50, C51, C52, C53, C54, C55, C56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

Commit message: done pcb layout
Other:
- company: Ryan Di Lorenzo -> LimesKey
Changed lines of the file:
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@@
 		(title "Battery Charger / Battery Managment System (BMS)")
 		(date "2026-08-24")
-		(company "Ryan Di Lorenzo")
+		(company "LimesKey")
 	)
 	(rectangle

Commit message: progress in layout!
Parts:
- R41: footprint Resistor_SMD:R_0805_2012Metric_Pad1.20x1.40mm_HandSolder -> footprints:R_Shunt_0805_2012Metric_Kelvin
- TP3: footprint TestPoint:TestPoint_Pad_D1.5mm -> TestPoint:TestPoint_Pad_D1.0mm; now left out of the parts list
Connections:
- net PMID: now reaches C80.1, C82.2, C86.2, C87.2, C88.2, U8.29 (PMID)
- net at Q5.8 (D), Q6.5 (D): now also Q5.5 (D), Q5.6 (D), Q5.7 (D), Q6.6 (D), Q6.7 (D), Q6.8 (D)
Changed lines of the file:
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@@
 	)
 	(junction
+		(at 148.59 132.08)
+		(diameter 0)
+		(color 0 0 0 0)
+	)
+	(junction
 		(at 52.07 184.15)
 		(diameter 0)
@@
 	)
 	(junction
+		(at 148.59 139.7)
+		(diameter 0)
+		(color 0 0 0 0)
+	)
+	(junction
 		(at 147.32 152.4)
 		(diameter 0)
@@
 	)
 	(junction
+		(at 148.59 137.16)
+		(diameter 0)
+		(color 0 0 0 0)
+	)
+	(junction
 		(at 78.74 158.75)
 		(diameter 0)
@@
 	)
 	(junction
+		(at 148.59 134.62)
+		(diameter 0)
+		(color 0 0 0 0)
+	)
+	(junction
 		(at 149.86 184.15)
 		(diameter 0)
@@
 	(wire
 		(pts
+			(xy 148.59 139.7) (xy 149.86 139.7)
+		)
+		(stroke
+			(width 0)
+			(type default)
+		)
+	)
+	(wire
+		(pts
 			(xy 162.56 105.41) (xy 168.91 105.41)
 		)
@@
 	(wire
 		(pts
+			(xy 148.59 137.16) (xy 149.86 137.16)
+		)
+		(stroke
+			(width 0)
+			(type default)
+		)
+	)
+	(wire
+		(pts
 			(xy 173.99 105.41) (xy 173.99 104.14)
 		)
@@
 	(wire
 		(pts
+			(xy 148.59 132.08) (xy 149.86 132.08)
+		)
+		(stroke
+			(width 0)
+			(type default)
+		)
+	)
+	(wire
+		(pts
 			(xy 275.59 82.55) (xy 275.59 83.82)
 		)
@@
 	(wire
 		(pts
-			(xy 146.05 139.7) (xy 149.86 139.7)
+			(xy 146.05 139.7) (xy 148.59 139.7)
 		)
 		(stroke
@@
 	(wire
 		(pts
-			(xy 146.05 137.16) (xy 149.86 137.16)
+			(xy 146.05 137.16) (xy 148.59 137.16)
 		)
 		(stroke
@@
 	(wire
 		(pts
+			(xy 148.59 134.62) (xy 149.86 134.62)
+		)
+		(stroke
+			(width 0)
+			(type default)
+		)
+	)
+	(wire
+		(pts
+			(xy 148.59 134.62) (xy 148.59 137.16)
+		)
+		(stroke
+			(width 0)
+			(type default)
+		)
+	)
+	(wire
+		(pts
 			(xy 52.07 186.69) (xy 57.15 186.69)
 		)
@@
 	(wire
 		(pts
+			(xy 148.59 137.16) (xy 148.59 139.7)
+		)
+		(stroke
+			(width 0)
+			(type default)
+		)
+	)
+	(wire
+		(pts
 			(xy 163.83 45.72) (xy 165.1 45.72)
 		)
@@
 	(wire
 		(pts
-			(xy 146.05 132.08) (xy 149.86 132.08)
+			(xy 146.05 132.08) (xy 148.59 132.08)
 		)
 		(stroke
@@
 	(wire
 		(pts
-			(xy 146.05 134.62) (xy 149.86 134.62)
+			(xy 146.05 134.62) (xy 148.59 134.62)
 		)
 		(stroke
@@
 	(wire
 		(pts
+			(xy 148.59 132.08) (xy 148.59 134.62)
+		)
+		(stroke
+			(width 0)
+			(type default)
+		)
+	)
+	(wire
+		(pts
 			(xy 110.49 137.16) (xy 120.65 137.16)
 		)
@@
 		)
 	)
+	(label "PMID"
+		(at 233.68 45.72 0)
+		(effects
+			(font
+				(size 1.27 1.27)
+			)
+			(justify left bottom)
+		)
+	)
 	(global_label "I2C_HOST_SDA"
 		(shape bidirectional)
@@
 			)
 		)
-		(property "Footprint" "Resistor_SMD:R_0805_2012Metric_Pad1.20x1.40mm_HandSolder"
+		(property "Footprint" "footprints:R_Shunt_0805_2012Metric_Kelvin"
 			(at 62.23 185.928 90)
 			(hide yes)
@@
 		(body_style 1)
 		(exclude_from_sim no)
-		(in_bom yes)
+		(in_bom no)
 		(on_board yes)
 		(in_pos_files yes)
@@
 			)
 		)
-		(property "Footprint" "TestPoint:TestPoint_Pad_D1.5mm"
+		(property "Footprint" "TestPoint:TestPoint_Pad_D1.0mm"
 			(at 127 179.07 0)
 			(hide yes)
