File: parsnip.kicad_sch (KiCad schematic)
At the start: 17 parts, among them J1 I2C1, J2 SPI BUS, J7 I2C2, J8 GCT USB4105-GF-A-120, U7 ESP32-S3-WROOM-1

Commit message: rename sheets, add lora antenna detect, seperate charger and regulator schematics, add eFuse to 5v output
Parts:
- added C131: 10uF, symbol Device:C_Small
- added C25: 1uF, Capacitor_SMD:C_0402_1005Metric, symbol Device:C_Small
Connections:
- net +3V3: now also U7.2 (3V3), C131.1, C25.1
- net GND: now also C131.2, C25.2
Other:
- sheet LORA renamed LoRa
- removed sheet Power_Management
- sheet GNSS: file GNSS-NEO.kicad_sch -> gnss.kicad_sch
- sheet LoRa: file LORA-E22.kicad_sch -> lora.kicad_sch

Commit message: Reworking power rails, adding antenna detection, and organization
Parts:
- removed J8: GCT USB4105-GF-A-120, Connector_USB:USB_C_Receptacle_GCT_USB4105-xx-A_16P_TopMnt_Horizontal, symbol Connector:USB_C_Receptacle_USB2.0_16P
Connections:
- net GND: now also U7.1 (GND), U7.40 (GND), U7.41 (GND)
Changed lines of the file:
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@@
 	(wire
 		(pts
+			(xy 62.23 167.64) (xy 62.23 170.18)
+		)
+		(stroke
+			(width 0)
+			(type default)
+		)
+	)
+	(wire
+		(pts
 			(xy 34.29 111.76) (xy 52.07 111.76)
 		)
@@
 	)
 	(symbol
-		(lib_id "Connector:USB_C_Receptacle_USB2.0_16P")
-		(at 146.05 62.23 0)
+		(lib_id "power:GND")
+		(at 62.23 170.18 0)
 		(unit 1)
 		(body_style 1)
@@
 		(in_pos_files yes)
 		(dnp no)
-		(fields_autoplaced yes)
-		(property "Reference" "J8"
-			(at 146.05 39.37 0)
-			(show_name no)
-			(do_not_autoplace no)
-			(effects
-				(font
-					(size 1.27 1.27)
-				)
-			)
-		)
-		(property "Value" "GCT USB4105-GF-A-120"
-			(at 146.05 41.91 0)
-			(show_name no)
-			(do_not_autoplace no)
-			(effects
-				(font
-					(size 1.27 1.27)
-				)
-			)
-		)
-		(property "Footprint" "Connector_USB:USB_C_Receptacle_GCT_USB4105-xx-A_16P_TopMnt_Horizontal"
-			(at 149.86 62.23 0)
+		(property "Reference" "#PWR0119"
+			(at 62.23 176.53 0)
 			(hide yes)
 			(show_name no)
@@
 			)
 		)
-		(property "Datasheet" "https://gct.co/files/drawings/usb4105.pdf"
-			(at 149.86 62.23 0)
-			(hide yes)
-			(show_name no)
-			(do_not_autoplace no)
-			(effects
-				(font
-					(size 1.27 1.27)
-				)
-			)
-		)
-		(property "Description" "USB 2.0-only 16P Type-C Receptacle connector"
-			(at 146.05 62.23 0)
-			(hide yes)
+		(property "Value" "GND"
+			(at 62.23 174.498 0)
 			(show_name no)
 			(do_not_autoplace no)
@@
 			)
 		)
-		(property "LCSC Part" "C5184243"
-			(at 146.05 62.23 0)
+		(property "Footprint" ""
+			(at 62.23 170.18 0)
 			(hide yes)
 			(show_name no)
@@
 			)
 		)
-		(property "Voltage Rating" ""
-			(at 146.05 62.23 0)
+		(property "Datasheet" ""
+			(at 62.23 170.18 0)
 			(hide yes)
 			(show_name no)
@@
 			)
 		)
-		(property "Tolerance" ""
-			(at 146.05 62.23 0)
+		(property "Description" "Power symbol creates a global label with name \"GND\" , ground"
+			(at 62.23 170.18 0)
 			(hide yes)
 			(show_name no)
@@
 			)
 		)
-		(pin "B6"
-		)
-		(pin "A8"
-		)
-		(pin "B1"
-		)
-		(pin "A7"
-		)
-		(pin "A9"
-		)
-		(pin "SH"
-		)
-		(pin "B7"
-		)
-		(pin "A5"
-		)
-		(pin "B9"
-		)
-		(pin "B8"
-		)
-		(pin "B12"
-		)
-		(pin "B5"
-		)
-		(pin "B4"
-		)
-		(pin "A4"
-		)
-		(pin "A1"
-		)
-		(pin "A12"
-		)
-		(pin "A6"
+		(pin "1"
 		)
 		(instances
 			(project "parsnip"
 				(path "/fe9d4a31-2311-442f-997c-52ad8ca5cfe9"
-					(reference "J8")
+					(reference "#PWR0119")
 					(unit 1)
 				)
@@
 			(project "parsnip"
 				(path "/fe9d4a31-2311-442f-997c-52ad8ca5cfe9"
-					(page "6")
+					(page "4")
 				)
 			)
@@
 			(project "parsnip"
 				(path "/fe9d4a31-2311-442f-997c-52ad8ca5cfe9"
-					(page "7")
+					(page "5")
 				)
 			)
@@
 		)
 	)
+	(embedded_fonts no)
 )

Commit message: usb-org
Parts:
- added C150: 10uF, symbol Device:C_Small
- added C151: 1uF, symbol Device:C_Small
- added C152, C153: 100nF, Capacitor_SMD:C_0402_1005Metric, symbol Device:C_Small
- added R100, R101, R98, R99: 0, Resistor_SMD:R_0402_1005Metric, symbol Device:R_Small
- added R97: 10k, symbol Device:R_Small
- added SW4: ESP_RESET, symbol Switch:SW_Push
- added SW5: BOOT, symbol Switch:SW_Push
Connections:
- net +3V3: now also C150.1, R97.1
- net GND: now also C150.2, C151.1, C152.1, C153.1, SW4.1, SW5.1
- net at U7.13 (USB_D-): now also R98.1
- net at U7.14 (USB_D+): now also R99.1
- net BOOT: now reaches U7.27 (IO0)
- net BOOT: now also R101.2
- net EN: now reaches U7.3 (EN)
- net EN: now also C151.2, R100.2, R97.2
- new net: C153.2, R101.1, SW5.2
- new net: C152.2, R100.1, SW4.2
- new net C_USB_B_N: R98.2
- new net C_USB_B_P: R99.2
Other:
- moved on the sheet: C131, C25, U7

Commit message: push to work on laptop2
Parts:
- added JP13: I2C_IRQ_PULLUP, Jumper:SolderJumper-2_P1.3mm_Bridged_RoundedPad1.0x1.5mm, symbol Jumper:SolderJumper_2_Bridged
- added JP14: I2C_SDA_PULLUP, Jumper:SolderJumper-2_P1.3mm_Bridged_RoundedPad1.0x1.5mm, symbol Jumper:SolderJumper_2_Bridged
- added JP15: I2C_SCL_PULLUP, Jumper:SolderJumper-2_P1.3mm_Bridged_RoundedPad1.0x1.5mm, symbol Jumper:SolderJumper_2_Bridged
- added R102: 10k, Resistor_SMD:R_0402_1005Metric_Pad0.72x0.64mm_HandSolder, symbol Device:R_Small
- added R103, R104: 2.2k, Resistor_SMD:R_0402_1005Metric_Pad0.72x0.64mm_HandSolder, symbol Device:R_Small
- added R105, R106: 22, Resistor_SMD:R_0402_1005Metric_Pad0.72x0.64mm_HandSolder, symbol Device:R_Small
- added R107, R108: 0, Resistor_SMD:R_0402_1005Metric, symbol Device:R_Small
- C27, C8, C9: value 10uF -> 2.2uF; Voltage Rating (none) -> 25V
Connections:
- net SCL_I2C is gone; now on net I2C_HOST_SCL: D4.1 (I/O1), J1.3 (Pin_3), J7.3 (Pin_3)
- net SDA_I2C is gone; now on net I2C_HOST_SDA: D4.3 (I/O2), J1.4 (Pin_4), J7.4 (Pin_4)
- net +3V3: now also R102.2, R103.2, R104.2
- net BUSY_LORA: now also U7.22 (IO14)
- net CS_LORA: now also U7.18 (IO10)
- net DIO1_LORA: now also U7.8 (IO15)
- net EN_LORA: now also U7.34 (IO41), R108.2
- net I2C_HOST_IRQ: now also U7.7 (IO7), JP13.1 (A)
- net I2C_HOST_SCL: now also U7.17 (IO9), JP15.1 (A)
- net I2C_HOST_SDA: now also U7.12 (IO8), JP14.1 (A)
- net MISO: now also U7.21 (IO13)
- net MOSI: now also R106.1
- net NRST_LORA: now also U7.33 (IO40), R107.1
- net SCK: now also R105.1
- net at U7.19 (IO11): now also R106.2
- net at U7.20 (IO12): now also R105.2
- net UART0_RX: now reaches U7.36 (RXD0)
- net UART0_TX: now reaches U7.37 (TXD0)
- net CS_BUS: no longer names the net of J2.6 (Pin_6)
- net CS_BUS: no longer D5.5 (I/O4)
- net C_USB_B_N renamed USB D-
- net C_USB_B_P renamed USB D+
- new net: JP15.2 (B), R104.1
- new net: JP14.2 (B), R103.1
- new net: JP13.2 (B), R102.1
- new net LoRa/EN: R108.1
- new net LoRa/RESET: R107.2
- no-connect marks 1 -> 9
Other:
- sheet GNSS ports: added EXTINT, PG_GNSS, SDA/SPI_CS; removed SDA/SPI_SS
- company: (none) -> Ryan Di Lorenzo
- title: (none) -> MCU + GPIO
- moved on the sheet: C27, C8, C9, D4, D5, F2, J2

Commit message: push for review, minor changes
Parts:
- added C154, C155: 6pF, Capacitor_SMD:C_0402_1005Metric, symbol Device:C_Small
- added JP4, JP5: SolderJumper_2_Open, symbol Jumper:SolderJumper_2_Open
- added R113, R114, R115: 0, Resistor_SMD:R_0402_1005Metric, symbol Device:R_Small
- added Y1: 32.768KHz, Crystal:Crystal_SMD_3215-2Pin_3.2x1.5mm, symbol Device:Crystal
- C1: renamed from C151; value 1uF -> 100nF; footprint (none) -> Capacitor_SMD:C_0402_1005Metric
- renumbered C131 to C2, C150 to C3, C25 to C4, C152 to C5, C153 to C6, C27 to C7, D5 to D1, D4 to D2, F2 to F1, F4 to F2, H4 to H1, H3 to H2, H2 to H3, H1 to H4, J2 to J1, J7 to J2, J1 to J3, JP13 to JP1, JP14 to JP2, JP15 to JP3, R97 to R1, R104 to R10, R108 to R11, R107 to R12, R106 to R2, R105 to R3, R98 to R4, R99 to R5, R100 to R6, R101 to R7, R102 to R8, R103 to R9, SW4 to SW1, SW5 to SW2, U7 to U1
Connections:
- net GND: now also C154.1, C155.1
- net GNSS/SCL/SPI_CLK: now also JP5.2 (B)
- net GNSS/SDA/SPI_CS: now also JP4.2 (B)
- net I2C_HOST_SCL: now also JP5.1 (A)
- net I2C_HOST_SDA: now also JP4.1 (A)
- net GPIO_21: now reaches U1.23 (IO21)
- net GPIO_48: now reaches U1.25 (IO48)
- net GPIO_4: now reaches U1.4 (IO4)
- net at U1.9 (IO16): now also R114.2
- net BUSY_LORA renamed GPIO_14
- net DIO1_LORA: no longer names the net of U1.8 (IO15)
- net DIO1_LORA: now also R113.2
- net EN_LORA renamed GPIO_41
- net NRST_LORA renamed GPIO_40
- new net: C155.2, R113.1, R115.2, Y1.1
- new net: C154.2, R114.1, R115.1, Y1.2
- no-connect marks 9 -> 6
Other:
- added sheet Rails (rails.kicad_sch)
- moved on the sheet: C5, C6, C7, C8, C9, D2, F1, F2, F3, J1, J2, J3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
