File: parsnip.kicad_sch (KiCad schematic)
At the start: 47 parts, among them J1 SPI BUS, J2 I2C2, J3 I2C1, SW1 ESP_RESET, SW2 BOOT, U1 ESP32-S3-WROOM-1, Y1 32.768KHz

Commit message: e-ink
Parts:
- removed F1, F2, F3: Littelfuse 0805L050WR, Fuse:Fuse_0805_2012Metric, symbol Device:Polyfuse_Small
- added C156: 2.2uF, Capacitor_SMD:C_0402_1005Metric, symbol Device:C_Small
- added C157: 10uF, Capacitor_SMD:C_0805_2012Metric, symbol Device:C_Small
- added D17: ESDS314DBVR, Package_TO_SOT_SMD:SOT-23-5, symbol easyeda2kicad:ESDS314DBVR-TP
- added D18: RB531SM-30, Diode_SMD:D_SOD-523, symbol Device:D_Schottky_Small
- added F5, F6, F7, F8: 2A Hold, 4A Trip, Fuse:Fuse_0805_2012Metric, symbol Device:Polyfuse_Small
- added J10: e-Ink Display Connector, symbol Connector_Generic_MountingPin:Conn_01x08_MountingPin
- added R116, R117: 10, Resistor_SMD:R_0402_1005Metric, symbol Device:R_Small
- D1, D2: value TI ESDS314DBVR -> ESDS314DBVR
Connections:
- net +3V3: now also F5.2, F6.2, F7.2, F8.2; no longer D2.4 (I/O3), D2.5 (I/O4)
- net GND: now also C156.2, C157.2, D17.2 (GND), J10.7 (Pin_7), J10.MP (MountPin)
- net MOSI: now also D17.5 (I/O4), R117.2
- net SCK: now also D17.4 (I/O3), R116.1
- net at J2.1 (Pin_1): now also F6.1
- net at J1.1 (Pin_1): now also F8.1
- net CS_BUS: now reaches J1.6 (Pin_6)
- net CS_BUS: now also D1.5 (I/O4), U1.31 (IO38)
- net CS_DISPLAY: now reaches U1.10 (IO17)
- net CS_DISPLAY: now also D2.4 (I/O3), D17.3 (I/O2), J10.4 (Pin_4)
- net D/C_DISPLAY: now reaches U1.11 (IO18)
- net D/C_DISPLAY: now also D17.1 (I/O1), J10.3 (Pin_3)
- net BUSY_DISPLAY: now reaches U1.5 (IO5)
- net BUSY_DISPLAY: now also J10.1 (Pin_1)
- net RESET_DISPLAY: now reaches U1.6 (IO6)
- net RESET_DISPLAY: now also D2.5 (I/O4), J10.2 (Pin_2)
- net at J3.1 (Pin_1): now also F7.1
- net CS_LORA renamed GPIO_10
- new net: D18.1 (K), J10.8 (Pin_8)
- new net: C156.1, C157.1, D18.2 (A), F5.1
- new net: J10.5 (Pin_5), R116.2
- new net: J10.6 (Pin_6), R117.1
- no-connect marks 6 -> 10
Other:
- note added: "Connectors"
- moved on the sheet: C7, C8, C9, D1, D2, H1, H2, H3, H4, J1, J2, J3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

Commit message: journal update!
Parts:
- added C169: 2.2uF, Capacitor_SMD:C_0402_1005Metric, symbol Device:C_Small
- added C170: 100nF, Capacitor_SMD:C_0402_1005Metric, symbol Device:C_Small
- added C63: 1uF, Capacitor_SMD:C_0402_1005Metric, symbol Device:C_Small
- added J12: UART0, symbol Connector:Conn_01x03_Socket
- added R118: 10k, symbol Device:R_Small
- added R121, R124, R125: 33, Resistor_SMD:R_0402_1005Metric_Pad0.72x0.64mm_HandSolder, symbol Device:R_Small
- added R126: 100k, Resistor_SMD:R_0402_1005Metric_Pad0.72x0.64mm_HandSolder, symbol Device:R_Small
- added R127, R128, R130: 10k, Resistor_SMD:R_0402_1005Metric_Pad0.72x0.64mm_HandSolder, symbol Device:R_Small
- added R59: 22, Resistor_SMD:R_0402_1005Metric, symbol Device:R_Small
- added U16: QMC6309, easyeda2kicad:X1-WLB0808-4_L0.8-W0.8-P0.40-TL, symbol easyeda2kicad:QMC6309
- C1, C5, C6: Capacitor Rating (none) -> X7R; LCSC Part (none) -> C5142567; Voltage Rating (none) -> 50V
- C154, C155: value 6pF -> 7pF
- C2, C3: footprint (none) -> Capacitor_SMD:C_0805_2012Metric; Capacitor Rating (none) -> X7R; LCSC Part C7472976 -> C380347
- C4: Capacitor Rating (none) -> X7R; LCSC Part (none) -> C46614478; Voltage Rating 16V -> 25V
- C7, C8, C9: Capacitor Rating (none) -> X5R; LCSC Part (none) -> C6119765
- D18: value RB531SM-30 -> 1N5819WS; footprint Diode_SMD:D_SOD-523 -> Diode_SMD:D_SOD-323; LCSC Part C2766159 -> C191023
- F5: value 2A Hold, 4A Trip -> SMD0805B035TF; LCSC Part C6851467 -> C269103
- F6, F8: value 2A Hold, 4A Trip -> 1A Hold
- R115: value 0 -> 10M
- R116: value 10 -> 22
- R117: value 10 -> 33; footprint Resistor_SMD:R_0402_1005Metric -> Resistor_SMD:R_0402_1005Metric_Pad0.72x0.64mm_HandSolder
Connections:
- net +3V3: now also D18.2 (A), C169.2, C170.2, C63.1, R118.1, R126.2, R127.2, R128.2, U16.B1 (VDD); no longer F5.2
- net BOOT: now also R118.2
- net BUSY_DISPLAY: now also D17.3 (I/O2)
- net CS_BUS: now also R117.1, R128.1; no longer J1.6 (Pin_6)
- net CS_DISPLAY: now also R127.1; no longer D17.3 (I/O2)
- net GND: now also C169.1, C170.1, C63.2, J12.1 (Pin_1), R130.2, U16.A1 (VSS)
- net GPIO_10: now also R126.1
- net I2C_HOST_SCL: now also U16.A2 (SCL)
- net I2C_HOST_SDA: now also U16.B2 (SDA)
- net MISO: now also R121.1; no longer J1.5 (Pin_5)
- net MOSI: now also J10.6 (Pin_6), R124.1; no longer D17.5 (I/O4), J1.4 (Pin_4), R117.2
- net RESET_DISPLAY: now also R130.1
- net SCK: now also J10.5 (Pin_5), R125.1; no longer D17.4 (I/O3), J1.3 (Pin_3), R116.1
- net UART0_RX: now also D17.5 (I/O4), R116.1
- net UART0_TX: now also D17.4 (I/O3), R59.1
- net GPIO_47: now reaches U1.24 (IO47)
- net UART1_TX: now reaches U1.38 (IO2)
- net UART1_RX: now reaches U1.39 (IO1)
- net at D18.1 (K): now also F5.2; no longer J10.8 (Pin_8)
- net at C156.1, C157.1, F5.1: now also J10.8 (Pin_8); no longer D18.2 (A)
- net at R116.2: now also J12.3 (Pin_3); no longer J10.5 (Pin_5)
- new net: J1.3 (Pin_3), R125.2
- new net: J1.4 (Pin_4), R124.2
- new net: J1.5 (Pin_5), R121.2
- new net: J1.6 (Pin_6), R117.2
- new net: J12.2 (Pin_2), R59.2
- no-connect marks 10 -> 13
Other:
- sheet Rails ports: added EN_CLOCK, PGOOD_EFUSE; removed none
- note added: "Pull up/down"
- moved on the sheet: C1, C154, C155, C2, C3, C4, C5, C6, D17, JP1, JP2, JP3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

Commit message: pcb layout!
Parts:
- added C1: 2.2uF, Capacitor_SMD:C_0402_1005Metric, symbol Device:C_Small
- added C176: 1uF, Capacitor_SMD:C_0402_1005Metric, symbol Device:C_Small
- added C177: 10uF, Capacitor_SMD:C_0603_1608Metric, symbol Device:C_Small
- added J14: GPIO_Expander, Connector_PinSocket_2.54mm:PinSocket_2x08_P2.54mm_Horizontal, symbol Connector_Generic:Conn_02x08_Odd_Even
- added J2: I2C3, Connector_JST:JST_SH_SM04B-SRSS-TB_1x04-1MP_P1.00mm_Horizontal, symbol Connector_Generic:Conn_01x04
- added R133: 10k, Resistor_SMD:R_0402_1005Metric_Pad0.72x0.64mm_HandSolder, symbol Device:R_Small
- added U17: TCAL9539RTWR_C22445413, easyeda2kicad:TQFN-24_L4.0-W4.0-P0.50-BL-EP2.3, symbol easyeda2kicad:TCAL9539RTWR_C22445413
- C10: renamed from C2; footprint Capacitor_SMD:C_0805_2012Metric -> Capacitor_SMD:C_0603_1608Metric; LCSC Part C380347 -> C22392391
- C11: renamed from C3; footprint Capacitor_SMD:C_0805_2012Metric -> Capacitor_SMD:C_0603_1608Metric; LCSC Part C380347 -> C22392391
- C12: renamed from C4; LCSC Part C46614478 -> C53426846
- C13: renamed from C156; LCSC Part (none) -> C33546001
- C14: renamed from C157; LCSC Part C33546010 -> C6119892
- C15: renamed from C169; LCSC Part (none) -> C33546001
- C16: renamed from C170; LCSC Part C5142567 -> C5272680
- C17: renamed from C63; LCSC Part (none) -> C53426846
- C2: renamed from C9; LCSC Part C6119765 -> C33546001
- C3: renamed from C8; LCSC Part C6119765 -> C33546001
- C4: renamed from C5; LCSC Part C5142567 -> C5272680
- C5: renamed from C6; LCSC Part C5142567 -> C5272680
- C6: renamed from C155; LCSC Part (none) -> C2929131
- C7: renamed from C154; LCSC Part (none) -> C2929131
- C8: renamed from C7; LCSC Part C6119765 -> C33546001
- C9: renamed from C1; LCSC Part C5142567 -> C5272680
- F1: renamed from F8; LCSC Part C6851467 -> C135331
- F3: renamed from F6; LCSC Part C6851467 -> C135331
- J5: renamed from J10; footprint (none) -> Connector_Molex:Molex_PicoBlade_53261-0871_1x08-1MP_P1.25mm_Horizontal; LCSC Part (none) -> C3029365
- J6: renamed from J12; footprint (none) -> Connector_JST:JST_SH_SM03B-SRSS-TB_1x03-1MP_P1.00mm_Horizontal
- JP1: renamed from JP4; footprint (none) -> Jumper:SolderJumper-2_P1.3mm_Open_TrianglePad1.0x1.5mm
- JP2: renamed from JP5; footprint (none) -> Jumper:SolderJumper-2_P1.3mm_Open_TrianglePad1.0x1.5mm
- R1: renamed from R125; LCSC Part (none) -> C54530835
- R10: renamed from R2; LCSC Part (none) -> C2686485
- R11: renamed from R3; LCSC Part (none) -> C2686485
- R12: renamed from R113; LCSC Part (none) -> C844711
- R13: renamed from R114; LCSC Part (none) -> C844711
- R14: renamed from R4; LCSC Part (none) -> C844711
- R15: renamed from R5; LCSC Part (none) -> C844711
- R16: renamed from R59; LCSC Part (none) -> C2686485
- R17: renamed from R116; LCSC Part (none) -> C2686485
- R18: renamed from R11; LCSC Part (none) -> C844711
- R19: renamed from R12; LCSC Part (none) -> C844711
- R2: renamed from R124; LCSC Part (none) -> C54530835
- R20: renamed from R8; LCSC Part (none) -> C2902636
- R21: renamed from R9; LCSC Part (none) -> C23901508
- R22: renamed from R10; LCSC Part (none) -> C23901508
- R23: renamed from R126; LCSC Part (none) -> C2984406
- R24: renamed from R127; LCSC Part (none) -> C2902636
- R25: renamed from R128; LCSC Part (none) -> C2902636
- R26: renamed from R130; LCSC Part (none) -> C2902636
- R3: renamed from R121; LCSC Part (none) -> C54530835
- R4: renamed from R117; LCSC Part (none) -> C54530835
- R5: renamed from R6; LCSC Part (none) -> C844711
- R6: renamed from R7; LCSC Part (none) -> C844711
- R7: renamed from R118; footprint (none) -> Resistor_SMD:R_0402_1005Metric; LCSC Part (none) -> C2902636
- R8: renamed from R115; footprint Resistor_SMD:R_0402_1005Metric -> Resistor_SMD:R_0805_2012Metric; LCSC Part (none) -> C54102219
- R9: renamed from R1; footprint (none) -> Resistor_SMD:R_0402_1005Metric; LCSC Part (none) -> C2902636
- SW1, SW2: footprint (none) -> Button_Switch_SMD:SW_Push_SPST_NO_Alps_SKRK; LCSC Part (none) -> C2681476
- U1: LCSC Part (none) -> C2913202
- renumbered D17 to D3, D18 to D4, F7 to F2, F5 to F4, J2 to J4, JP1 to JP3, JP2 to JP4, JP3 to JP5, U16 to U2
Connections:
- net +3V3: now also C1.1, C176.1, C177.1, J2.2 (Pin_2), R133.2, U17.21 (VCC)
- net GND: now also C1.2, C176.2, C177.2, J14.14 (Pin_14), J14.16 (Pin_16), J2.1 (Pin_1), U17.18 (A0), U17.23 (A1), U17.25 (EP), U17.9 (GND)
- net I2C_HOST_IRQ: now also U17.22 (~{INT})
- net I2C_HOST_SCL: now also J2.3 (Pin_3), U17.19 (SCL)
- net I2C_HOST_SDA: now also J2.4 (Pin_4), U17.20 (SDA)
- net GPIO_3: now reaches U1.15 (IO3)
- net GPIO_39: now reaches U1.32 (IO39)
- net GPIO_42: now reaches U1.35 (IO42)
- new net: J14.1 (Pin_1), U17.1 (P00)
- new net: J14.3 (Pin_3), U17.2 (P01)
- new net: J14.5 (Pin_5), U17.3 (P02)
- new net: J14.7 (Pin_7), U17.4 (P03)
- new net: J14.9 (Pin_9), U17.5 (P04)
- new net: J14.11 (Pin_11), U17.6 (P05)
- new net: J14.13 (Pin_13), U17.7 (P06)
- new net: J14.15 (Pin_15), U17.8 (P07)
- new net IO_EXP_RESET: R133.1, U17.24 (~{RESET})
- new net P12: J14.2 (Pin_2), U17.12 (P12)
- new net P13: J14.4 (Pin_4), U17.13 (P13)
- new net P14: J14.6 (Pin_6), U17.14 (P14)
- new net P15: J14.8 (Pin_8), U17.15 (P15)
- new net P16: J14.10 (Pin_10), U17.16 (P16)
- new net P17: J14.12 (Pin_12), U17.17 (P17)
- no-connect marks 13 -> 5
Other:
- sheet LoRa ports: added none; removed TR_CTRL
- note added: "Magnetometer"
- moved on the sheet: C10, C11, C12, C17, C4, C5, C6, C7, C9, D1, D2, JP3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

Commit message: organize repo and schematic
Parts:
- removed C15: 2.2uF, Capacitor_SMD:C_0402_1005Metric, symbol Device:C_Small
- removed C16: 100nF, Capacitor_SMD:C_0402_1005Metric, symbol Device:C_Small
- removed C176: 1uF, Capacitor_SMD:C_0402_1005Metric, symbol Device:C_Small
- removed C177: 10uF, Capacitor_SMD:C_0603_1608Metric, symbol Device:C_Small
- removed J14: GPIO_Expander, Connector_PinSocket_2.54mm:PinSocket_2x08_P2.54mm_Horizontal, symbol Connector_Generic:Conn_02x08_Odd_Even
- removed U17: TCAL9539RTWR_C22445413, easyeda2kicad:TQFN-24_L4.0-W4.0-P0.50-BL-EP2.3, symbol easyeda2kicad:TCAL9539RTWR_C22445413
- removed U2: QMC6309, easyeda2kicad:X1-WLB0808-4_L0.8-W0.8-P0.40-TL, symbol easyeda2kicad:QMC6309
- U1: value ESP32-S3-WROOM-1 -> ESP32-S3-WROOM-1-N16R8
Connections:
- net GPIO_46: now reaches U1.16 (IO46)
- no-connect marks 5 -> 4
Other:
- added sheet Peripherals (peripherals.kicad_sch)
- note removed: "Magnetometer"
- moved on the sheet: C10, C11, C12, C4, C5, C6, C7, C9, R10, R11, R12, R13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

Commit message: done pcb layout
Parts:
- removed R133: 10k, Resistor_SMD:R_0402_1005Metric_Pad0.72x0.64mm_HandSolder, symbol Device:R_Small
- added TP15: GPIO_EXP_RESET, TestPoint:TestPoint_Pad_D1.0mm, symbol Connector:TestPoint_Probe
- J1: footprint Connector_PinSocket_2.54mm:PinSocket_1x06_P2.54mm_Horizontal -> easyeda2kicad:HDR-SMD_6P-P2.54-H-F-W11.7; LCSC Part (none) -> C46061770
- J3: footprint Connector_PinSocket_2.54mm:PinSocket_1x04_P2.54mm_Horizontal -> easyeda2kicad:CONN-SMD_4P-P2.54_HX-PM2.54-1X4PWT; LCSC Part (none) -> C46061768
Connections:
- net +3V3: now also JP3.2 (B), JP4.2 (B), JP5.2 (B); no longer R20.2, R21.2, R22.2
- net I2C_HOST_IRQ: now also R20.1; no longer JP3.1 (A)
- net I2C_HOST_SCL: now also R22.1; no longer JP5.1 (A)
- net I2C_HOST_SDA: now also R21.1; no longer JP4.1 (A)
- new net: JP5.1 (A), R22.2
- new net: JP3.1 (A), R20.2
- new net: JP4.1 (A), R21.2
- new net Peripherals/RESET_IOEXP: TP15.1
Other:
- sheet Peripherals ports: added IO_P16, IO_P17, LED_DIN, RESET_IOEXP; removed none
- note added: "Connectors/Pin Headers"
- note removed: "Connectors"
- company: Ryan Di Lorenzo -> LimesKey
- moved on the sheet: C17, C4, R26, R5, SW1

Commit message: progress in layout!
Parts:
- removed C4, C9: 100nF, Capacitor_SMD:C_0402_1005Metric, symbol Device:C_Small
- added C182: 1uF, Capacitor_SMD:C_0402_1005Metric, symbol Device:C_Small
- TP15: footprint TestPoint:TestPoint_Pad_D1.0mm -> TestPoint:TestPoint_Pad_D1.5mm
Connections:
- net GND: now also C6.2, C182.1; no longer C6.1
- net at R12.1, R8.2, Y1.1: now also C6.1; no longer C6.2
- net at R5.1, SW1.2: now also C182.2
Other:
- moved on the sheet: C10, C11, C12, C5, R10, R11, R12, R13, R14, R15, R5, R6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
