File: usb_interface.kicad_sch (KiCad schematic)
At the start: 51 parts, among them J8 GCT USB4105-GF-A-120, J9 PD_I2C DEBUG, Q10 CSD15380F3, Q6 CSD25480F3, Q8 CSD15380F3, Q9 CSD25480F3, U1 CAT24C256, U12 TI TPS25751DREFR, U14 TVS2200DRV, U4 TPD8S300A

Commit message: push to work on laptop2
Parts:
- removed D19: TPD4E05U06DQAR_C138714, easyeda2kicad:USON-10_L2.5-W1.0-P0.50-BL, symbol easyeda2kicad:TPD4E05U06DQAR_C138714
- added NT5, NT6: NetTie_3, NetTie:NetTie-3_SMD_Pad0.5mm, symbol Device:NetTie_3
- U4: value TPD8S300A -> TPD8S300/A; LCSC Part C2649824 -> C571205
Connections:
- net C_CC1: now also U4.7 (RPD_G1)
- net C_CC2: now also U4.6 (RPD_G2)
- net C_USB_B_N: now also NT5.3
- net C_USB_B_P: now also NT6.3
- net C_USB_T_N: now also NT5.1
- net C_USB_T_P: now also NT6.1
- net GND: no longer U4.6 (RPD_G2), U4.7 (RPD_G1)
- new net USB D+: NT6.2
- new net USB D-: NT5.2
Other:
- title: (none) -> USB Interface

Commit message: push for review, minor changes
Parts:
- renumbered C146 to C10, C142 to C11, C143 to C12, C144 to C13, C145 to C14, C147 to C15, C41 to C16, C32 to C17, C7 to C18, C29 to C19, C6 to C20, C26 to C21, C1 to C22, C12 to C23, C67 to C24, C5 to C25, C78 to C26, C83 to C27, C135 to C28, C136 to C29, C95 to C30, C99 to C31, C112 to C32, C113 to C33, C149 to C34, C114 to C35, C148 to C36, J8 to J4, J9 to J5, JP12 to JP6, NT5 to NT1, NT6 to NT2, Q6 to Q1, Q10 to Q2, Q9 to Q3, Q8 to Q4, R92 to R13, R60 to R14, R90 to R15, R91 to R16, R89 to R17, R86 to R18, R88 to R19, R93 to R20, R96 to R21, R94 to R22, R95 to R23, U14 to U2, U4 to U3, U12 to U4, U1 to U5
Connections:
- net GND: no longer U4.6 (GPIO1)
- net I2C_HOST_IRQ: now also U4.6 (GPIO1)
