File: usb_interface.kicad_sch (KiCad schematic)
At the start: 52 parts, among them J4 GCT USB4105-GF-A-120, J5 PD_I2C DEBUG, Q1 CSD25480F3, Q2 CSD15380F3, Q3 CSD25480F3, Q4 CSD15380F3, U2 TVS2200DRV, U3 TPD8S300/A, U4 TI TPS25751DREFR, U5 CAT24C256

Commit message: journal update!
Parts:
- removed JP6: WRITE_PROTECT, Jumper:SolderJumper-2_P1.3mm_Bridged_RoundedPad1.0x1.5mm, symbol Jumper:SolderJumper_2_Bridged
- added C166, C69: 10uF, Capacitor_SMD:C_1206_3216Metric, symbol Device:C_Small
- added JP17: WRITE_PROTECT, symbol Jumper:SolderJumper_3_Bridged12
- added R129: 10k, Resistor_SMD:R_0402_1005Metric, symbol Device:R_Small
- C10: Capacitor Rating (none) -> X5R; LCSC Part C23692972 -> C46614478; Voltage Rating 16V -> 25V
- C12, C13, C14: Voltage Rating (none) -> 50V
- C16: Voltage Rating 100V -> 50V
- C17, C18, C19, C21, C23: footprint Capacitor_SMD:C_1206_3216Metric -> Capacitor_SMD:C_1210_3225Metric
- C20: value 2.2uF -> 4.7uF; footprint Capacitor_SMD:C_0603_1608Metric -> Capacitor_SMD:C_1206_3216Metric
- C34, C36: Voltage Rating 50V -> 16V
- C35: value 100nF -> 1uF
Connections:
- net GND: now also C166.2, C69.1; no longer U4.19 (GPIO3)
- net PD_LDO_3V3: now also Q1.2 (S), Q3.2 (S), R129.2; no longer Q1.3 (D), Q3.3 (D)
- net PPHV: now also C166.1, C69.2
- net WC: now also JP17.2 (C)
- net at R22.1: now also Q3.3 (D); no longer Q3.2 (S)
- net FAULT: now reaches R13.2, U3.9 (~{FLT})
- net FAULT: now also U4.19 (GPIO3)
- net at RN1.5 (R4): now also JP17.1 (A)
- net at R20.1: now also Q1.3 (D); no longer Q1.2 (S)
- new net: JP17.3 (B), R129.1
Other:
- note added: "8 x 10uF"
- note added: "EEPROM 256Kb"
- note removed: "6 x 10uF"
- moved on the sheet: C17, C18, C19, C21, C23, C34, C35, C36, J5, Q1, Q2, Q3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

Commit message: pcb layout!
Parts:
- removed RN1: 10k, Resistor_SMD:R_Array_Concave_4x0402, symbol Device:R_Network04
- added RN1: 10k, Resistor_SMD:R_Array_Concave_4x0402, symbol Device:R_Pack04
- C18: renamed from C10; LCSC Part C46614478 -> C53426846
- C19: renamed from C11; footprint (none) -> Capacitor_SMD:C_0402_1005Metric; Capacitor Rating (none) -> X7R; LCSC Part (none) -> C5272680
- C20: renamed from C34; LCSC Part (none) -> C53426846
- C21: renamed from C12; LCSC Part (none) -> C696856
- C22: renamed from C13; LCSC Part (none) -> C696856
- C23: renamed from C14; LCSC Part (none) -> C696856
- C24: renamed from C15; footprint (none) -> Capacitor_SMD:C_0402_1005Metric; Capacitor Rating (none) -> X7R; LCSC Part (none) -> C5272680
- C25: renamed from C36; LCSC Part (none) -> C53426846
- C26: renamed from C16; footprint Capacitor_SMD:C_1210_3225Metric -> Capacitor_SMD:C_1206_3216Metric; LCSC Part C5156756 -> C14860
- C27: renamed from C166; LCSC Part C33546013 -> C49326770
- C28: renamed from C69; LCSC Part C33546013 -> C49326770
- C29: renamed from C17; footprint Capacitor_SMD:C_1210_3225Metric -> Capacitor_SMD:C_1206_3216Metric; LCSC Part C33546013 -> C14860
- C30: renamed from C18; footprint Capacitor_SMD:C_1210_3225Metric -> Capacitor_SMD:C_1206_3216Metric; LCSC Part C33546013 -> C14860
- C31: renamed from C20; footprint Capacitor_SMD:C_1206_3216Metric -> Capacitor_SMD:C_0805_2012Metric; LCSC Part (none) -> C7472970
- C32: renamed from C19; footprint Capacitor_SMD:C_1210_3225Metric -> Capacitor_SMD:C_1206_3216Metric; LCSC Part C33546013 -> C14860
- C33: renamed from C22; footprint (none) -> Capacitor_SMD:C_0402_1005Metric; LCSC Part (none) -> C190579
- C34: renamed from C21; footprint Capacitor_SMD:C_1210_3225Metric -> Capacitor_SMD:C_1206_3216Metric; LCSC Part C33546013 -> C14860
- C35: renamed from C23; footprint Capacitor_SMD:C_1210_3225Metric -> Capacitor_SMD:C_1206_3216Metric; LCSC Part C33546013 -> C14860
- C36: renamed from C25; footprint (none) -> Capacitor_SMD:C_0402_1005Metric; LCSC Part (none) -> C190579
- C38: renamed from C26; LCSC Part (none) -> C6119892
- C39: renamed from C27; LCSC Part C23692972 -> C53426846
- C40: renamed from C28; LCSC Part (none) -> C6119892
- C41: renamed from C29; LCSC Part C23692972 -> C53426846
- C42: renamed from C30; LCSC Part (none) -> C6119892
- C43: renamed from C31; LCSC Part C23692972 -> C53426846
- C44: renamed from C32; LCSC Part (none) -> C6119892
- C45: renamed from C33; LCSC Part C23692972 -> C53426846
- C46: renamed from C35; LCSC Part (none) -> C53426846
- J7: renamed from J4; LCSC Part C5184243 -> C3025063
- J8: renamed from J5; footprint (none) -> Connector_PinSocket_2.54mm:PinSocket_1x04_P2.54mm_Vertical
- JP6: renamed from JP17; footprint (none) -> Jumper:SolderJumper-3_P1.3mm_Bridged12_RoundedPad1.0x1.5mm_NumberLabels
- Q1, Q3: LCSC Part (none) -> C2869359
- Q2, Q4: footprint (none) -> Package_DFN_QFN:Texas_PicoStar_DFN-3_0.69x0.60mm; LCSC Part (none) -> C529568
- R27: renamed from R13; LCSC Part (none) -> C2984406
- R28: renamed from R20; LCSC Part (none) -> C2984406
- R29: renamed from R21; LCSC Part (none) -> C2918201
- R30: renamed from R22; LCSC Part (none) -> C2984406
- R31: renamed from R23; LCSC Part (none) -> C2918201
- R32: renamed from R14; LCSC Part (none) -> C844711
- R33: renamed from R15; LCSC Part (none) -> C844711
- R34: renamed from R16; LCSC Part (none) -> C844711
- R35: renamed from R17; footprint (none) -> Resistor_SMD:R_0402_1005Metric; LCSC Part (none) -> C2902636
- R36: renamed from R18; footprint (none) -> Resistor_SMD:R_0402_1005Metric; LCSC Part (none) -> C23901508
- R37: renamed from R19; footprint (none) -> Resistor_SMD:R_0402_1005Metric; LCSC Part (none) -> C23901508
- R38: renamed from R129; LCSC Part (none) -> C2902636
- renumbered C24 to C37, U2 to U3, U3 to U4, U4 to U5, U5 to U6
Connections:
- net GND: now also RN1.1 (R1.1), RN1.2 (R2.1), RN1.3 (R3.1), RN1.4 (R4.1)
- net at U6.3 (A2): now also RN1.5 (R4.2)
- net at U6.2 (A1): now also RN1.6 (R3.2)
- net at U6.1 (A0): now also RN1.7 (R2.2)
- net at JP6.1 (A): now also RN1.8 (R1.2)

Commit message: done pcb layout
Parts:
- added C184: 100nF, Capacitor_SMD:C_0402_1005Metric, symbol Device:C_Small
Connections:
- net GND: now also C184.2
- net VBUS: now also C184.1
Other:
- company: Ryan Di Lorenzo -> LimesKey
- moved on the sheet: C31, C33, C36

Commit message: add 3d models locally
Parts:
- U6: footprint Package_DFN_QFN:OnSemi_UDFN-8_1.2x1.8mm_P0.4mm -> Package_DFN_QFN:DFN-8-1EP_2x3mm_P0.5mm_EP0.61x2.2mm
Changed lines of the file:
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@@
 			)
 		)
-		(property "Footprint" "Package_DFN_QFN:OnSemi_UDFN-8_1.2x1.8mm_P0.4mm"
+		(property "Footprint" "Package_DFN_QFN:DFN-8-1EP_2x3mm_P0.5mm_EP0.61x2.2mm"
 			(at 243.84 90.17 0)
 			(hide yes)
