File: parsnip.kicad_pcb (KiCad board)
At the start: 4 copper layers, 55 x 100 mm, 93 parts, among them J1 I2C1, J2 SPI BUS, J3 Conn_Coaxial, J4 Conn_Coaxial_Small, J5 Conn_Coaxial, J6 Conn_01x02, J7 I2C2, Q1 AO3401A, Q3 CSD16301Q2, Q4 CSD16301Q2, SW1 SW_Push, U1 XIAO-ESP32-C6-SMD, U2 NEO-M9N, U3 E22P-915M30S, U4 BQ29700, U6 TPS2116DRL, U7 TPS61033DRLR

Commit message: pcb layout!
Parts:
- added BT2: 21700 Li-ion, easyeda2kicad:BAT-SMD_L82.5.5-W25-BH-21700-B1BJ001, B.Cu at (117.3, 53.5)
- added BT3: MS621FE 5.5mAh, Battery:BatteryHolder_Seiko_MS621F, F.Cu at (108.6, 39.0)
- added C100: 100nF, Capacitor_SMD:C_0402_1005Metric, F.Cu at (168.2, 72.3)
- added C101: 4.7uF, Capacitor_SMD:C_0402_1005Metric, F.Cu at (173.9, 47.8)
- added C102: 10uF, Capacitor_SMD:C_0402_1005Metric, F.Cu at (173.9, 49.8)
- added C103: 1uF, Capacitor_SMD:C_0402_1005Metric, F.Cu at (173.9, 51.8)
- added C104: 2.2uF, Capacitor_SMD:C_0402_1005Metric, F.Cu at (173.9, 53.7)
- added C105: 2.2uF, Capacitor_SMD:C_0402_1005Metric, F.Cu at (178.1, 46.5)
- added C106: 10uF, Capacitor_SMD:C_0402_1005Metric, F.Cu at (178.1, 49.9)
- added C107: 100nF, Capacitor_SMD:C_0402_1005Metric, F.Cu at (173.9, 55.7)
- added C108: 2.2nF, Capacitor_SMD:C_0402_1005Metric, F.Cu at (163.6, 122.5)
- added C109: 2.2nF, Capacitor_SMD:C_0402_1005Metric, F.Cu at (182.9, 145.2)
- added C110: 10uF, Capacitor_SMD:C_0603_1608Metric, F.Cu at (162.2, 145.3)
- added C111: 10uF, Capacitor_SMD:C_0402_1005Metric, F.Cu at (182.9, 147.7)
- added C112: 1nF, Capacitor_SMD:C_0402_1005Metric, F.Cu at (163.6, 125.9)
- added C113: 1pF, Capacitor_SMD:C_0402_1005Metric_Pad0.74x0.62mm_HandSolder, F.Cu at (182.9, 150.2)
- added C114: 1pF, Capacitor_SMD:C_0402_1005Metric_Pad0.74x0.62mm_HandSolder, F.Cu at (162.2, 147.3)
- added C115: 47pF, Capacitor_SMD:C_0402_1005Metric, F.Cu at (182.9, 152.8)
- added C116: 100nF, Capacitor_SMD:C_0402_1005Metric, F.Cu at (162.2, 149.2)
- added C117: 1uF, Capacitor_SMD:C_0402_1005Metric, F.Cu at (123.5, 44.4)
- added C118: 1uF, Capacitor_SMD:C_0402_1005Metric, F.Cu at (123.5, 46.3)
- added C119: 22uF, Capacitor_SMD:C_1206_3216Metric, F.Cu at (120.7, 44.8)
- added C120: 22uF, Capacitor_SMD:C_1206_3216Metric, F.Cu at (120.7, 47.3)
- added C121: 100nF, Capacitor_SMD:C_0402_1005Metric, F.Cu at (182.9, 155.3)
- added C122: 10uF, Capacitor_SMD:C_1206_3216Metric, F.Cu at (165.0, 145.3)
- added C123: 1uF, Capacitor_SMD:C_0603_1608Metric, F.Cu at (165.0, 147.3)
- added C124: 100nF, Capacitor_SMD:C_0402_1005Metric, F.Cu at (165.0, 149.2)
- added C125: 2.2uF, Capacitor_SMD:C_0603_1608Metric, F.Cu at (199.5, 156.9)
- added C126: 10uF, Capacitor_SMD:C_1206_3216Metric, F.Cu at (165.0, 151.2)
- added C127: 1uF, Capacitor_SMD:C_0603_1608Metric, F.Cu at (163.6, 129.2)
- added C128: 100nF, Capacitor_SMD:C_0402_1005Metric, F.Cu at (187.0, 145.2)
- added C129: 2.2uF, Capacitor_SMD:C_0603_1608Metric, F.Cu at (163.6, 132.6)
- added C130: 100nF, Capacitor_SMD:C_0402_1005Metric, F.Cu at (163.6, 135.9)
- added C131: 100nF, Capacitor_SMD:C_0402_1005Metric, F.Cu at (187.0, 147.7)
- added C132: 1uF, Capacitor_SMD:C_0402_1005Metric, F.Cu at (165.0, 153.2)
- added C133: 220pF, Capacitor_SMD:C_0402_1005Metric_Pad0.74x0.62mm_HandSolder, F.Cu at (165.0, 155.2)
- added C134: 100nF, Capacitor_SMD:C_0402_1005Metric, F.Cu at (163.6, 139.3)
- added C135: 2.2uF, Capacitor_SMD:C_0603_1608Metric, F.Cu at (163.6, 142.6)
- added C136: 100nF, Capacitor_SMD:C_0402_1005Metric, F.Cu at (169.2, 122.5)
- added C137: 1uF, Capacitor_SMD:C_0402_1005Metric, F.Cu at (187.0, 150.2)
- added C138: 1uF, Capacitor_SMD:C_0402_1005Metric, F.Cu at (199.5, 158.8)
- added C139: 220pF, Capacitor_SMD:C_0402_1005Metric_Pad0.74x0.62mm_HandSolder, F.Cu at (169.2, 125.9)
- added C140: 1uF, Capacitor_SMD:C_0402_1005Metric, F.Cu at (169.2, 129.2)
- added C141: 10uF, Capacitor_SMD:C_1206_3216Metric, F.Cu at (167.9, 145.3)
- added C142: 10uF, Capacitor_SMD:C_0603_1608Metric, F.Cu at (199.5, 160.8)
- added C143: 10uF, Capacitor_SMD:C_1206_3216Metric, F.Cu at (167.9, 147.3)
- added C144: 22uF, Capacitor_SMD:C_1206_3216Metric, F.Cu at (167.9, 149.2)
- added C145: 2.2uF, Capacitor_SMD:C_0603_1608Metric, F.Cu at (169.2, 132.6)
- added C146: 1uF, Capacitor_SMD:C_0402_1005Metric, F.Cu at (169.2, 135.9)
- added C147: 1uF, Capacitor_SMD:C_0402_1005Metric, F.Cu at (167.9, 151.2)
- added C148: 22uF, Capacitor_SMD:C_1206_3216Metric, F.Cu at (187.0, 152.8)
- added C149: 22uF, Capacitor_SMD:C_1206_3216Metric, F.Cu at (169.2, 139.3)
- added C150: 22uF, Capacitor_SMD:C_1206_3216Metric, F.Cu at (169.2, 142.6)
- added C151: 10uF, Capacitor_SMD:C_1206_3216Metric, F.Cu at (174.8, 122.5)
- added C152: 10uF, Capacitor_SMD:C_0603_1608Metric, F.Cu at (167.9, 153.2)
- added C153: 5.6pF, Capacitor_SMD:C_0402_1005Metric_Pad0.74x0.62mm_HandSolder, F.Cu at (174.8, 125.9)
- added C154: 10uF, Capacitor_SMD:C_1206_3216Metric, F.Cu at (195.3, 27.4)
- added C155: 22uF, Capacitor_SMD:C_1206_3216Metric, F.Cu at (195.3, 29.3)
- added C156: 1uF, Capacitor_SMD:C_0402_1005Metric, F.Cu at (195.3, 31.3)
- added C157: 1uF, Capacitor_SMD:C_0402_1005Metric, F.Cu at (192.8, 52.2)
- added C158: 5.6pF, Capacitor_SMD:C_0402_1005Metric_Pad0.74x0.62mm_HandSolder, F.Cu at (167.9, 155.2)
- added C159: 1nF, Capacitor_SMD:C_0402_1005Metric, F.Cu at (170.8, 145.3)
- added C160: 1nF, Capacitor_SMD:C_0402_1005Metric, F.Cu at (170.8, 147.3)
- added C161: 2.2nF, Capacitor_SMD:C_0402_1005Metric, F.Cu at (170.8, 149.2)
- added C162: 2.2nF, Capacitor_SMD:C_0402_1005Metric, F.Cu at (170.8, 151.2)
- added C163: 1uF, Capacitor_SMD:C_0402_1005Metric, F.Cu at (182.4, 27.5)
- added C164: 1uF, Capacitor_SMD:C_0402_1005Metric, F.Cu at (182.4, 30.8)
- added C165: 22uF, Capacitor_SMD:C_1206_3216Metric, F.Cu at (182.4, 34.2)
- added C166: 22uF, Capacitor_SMD:C_1206_3216Metric, F.Cu at (182.4, 37.5)
- added C167: 1uF, Capacitor_SMD:C_0402_1005Metric, F.Cu at (174.8, 129.2)
- added C168: 10uF, Capacitor_SMD:C_0603_1608Metric, F.Cu at (174.8, 132.6)
- added C169: 22uF, Capacitor_SMD:C_1206_3216Metric, F.Cu at (195.3, 33.3)
- added C170: 22uF, Capacitor_SMD:C_1206_3216Metric, F.Cu at (195.3, 35.2)
- added C171: 22uF, Capacitor_SMD:C_1206_3216Metric, F.Cu at (174.8, 135.9)
- added C172: 22uF, Capacitor_SMD:C_1206_3216Metric, F.Cu at (195.3, 37.2)
- added C173: 22uF, Capacitor_SMD:C_1206_3216Metric, F.Cu at (222.4, 85.8)
- added C174: 1uF, Capacitor_SMD:C_0402_1005Metric, F.Cu at (216.3, 81.9)
- added C175: 22uF, Capacitor_SMD:C_1206_3216Metric, F.Cu at (211.6, 85.8)
- added C176: 1uF, Capacitor_SMD:C_0402_1005Metric, F.Cu at (92.7, 97.7)
- added C177: 10uF, Capacitor_SMD:C_0603_1608Metric, F.Cu at (93.3, 93.4)
- added C28: 10uF, Capacitor_SMD:C_1206_3216Metric, F.Cu at (204.8, 47.8)
- added C29: 10uF, Capacitor_SMD:C_1206_3216Metric, F.Cu at (186.7, 23.4)
- added C30: 10uF, Capacitor_SMD:C_1206_3216Metric, F.Cu at (201.8, 47.8)
- added C31: 4.7uF, Capacitor_SMD:C_0805_2012Metric, F.Cu at (186.7, 25.4)
- added C32: 10uF, Capacitor_SMD:C_1206_3216Metric, F.Cu at (198.8, 47.8)
- added C33: 330pF, Capacitor_SMD:C_0402_1005Metric, F.Cu at (186.7, 27.4)
- added C34: 10uF, Capacitor_SMD:C_1206_3216Metric, F.Cu at (186.7, 29.3)
- added C35: 10uF, Capacitor_SMD:C_1206_3216Metric, F.Cu at (186.7, 31.3)
- added C36: 330pF, Capacitor_SMD:C_0402_1005Metric, F.Cu at (186.7, 33.3)
- added C37: 1uF, Capacitor_SMD:C_0603_1608Metric, F.Cu at (227.1, 96.7)
- added C38: 10uF, Capacitor_SMD:C_0805_2012Metric, F.Cu at (232.3, 91.6)
- added C39: 1uF, Capacitor_SMD:C_0402_1005Metric, F.Cu at (233.3, 101.5)
- added C40: 10uF, Capacitor_SMD:C_0805_2012Metric, F.Cu at (231.7, 71.2)
- added C41: 1uF, Capacitor_SMD:C_0402_1005Metric, F.Cu at (231.7, 73.1)
- added C42: 10uF, Capacitor_SMD:C_0805_2012Metric, F.Cu at (231.7, 75.1)
- added C43: 1uF, Capacitor_SMD:C_0402_1005Metric, F.Cu at (229.3, 103.5)
- added C44: 10uF, Capacitor_SMD:C_0805_2012Metric, F.Cu at (235.8, 87.5)
- added C45: 1uF, Capacitor_SMD:C_0402_1005Metric, F.Cu at (237.3, 106.0)
- added C46: 1uF, Capacitor_SMD:C_0402_1005Metric, F.Cu at (237.3, 104.0)
- added C47: 1uF, Capacitor_SMD:C_0402_1005Metric, F.Cu at (110.1, 99.8)
- added C48: 10uF, Capacitor_SMD:C_0805_2012Metric, B.Cu at (150.8, 110.2)
- added C49: 100nF, Capacitor_SMD:C_0402_1005Metric, F.Cu at (114.7, 99.5)
- added C50: 100nF, Capacitor_SMD:C_0402_1005Metric, F.Cu at (115.7, 97.5)
- added C51: 100nF, Capacitor_SMD:C_0402_1005Metric, F.Cu at (112.7, 99.5)
- added C52: 1uF, Capacitor_SMD:C_0402_1005Metric, F.Cu at (111.8, 101.0)
- added C53: 0.47uF, Capacitor_SMD:C_0402_1005Metric, F.Cu at (110.8, 101.8)
- added C54: 100nF, Capacitor_SMD:C_0402_1005Metric, F.Cu at (107.7, 104.5)
- added C55: 0.47uF, Capacitor_SMD:C_0402_1005Metric, F.Cu at (118.6, 104.0)
- added C56: 0.47uF, Capacitor_SMD:C_0402_1005Metric, F.Cu at (118.6, 102.0)
- added C57: 10uF, Capacitor_SMD:C_1206_3216Metric, F.Cu at (133.3, 76.7)
- added C58: 0.47uF, Capacitor_SMD:C_0402_1005Metric, F.Cu at (118.2, 107.1)
- added C59: 10uF, Capacitor_SMD:C_1206_3216Metric, F.Cu at (131.6, 74.2)
- added C60: 10uF, Capacitor_SMD:C_1206_3216Metric, F.Cu at (133.3, 79.4)
- added C61: 100nF, Capacitor_SMD:C_0402_1005Metric, F.Cu at (109.3, 106.0)
- added C62: 2.2uF, Capacitor_SMD:C_0805_2012Metric, F.Cu at (110.8, 90.0)
- added C63: 10uF, Capacitor_SMD:C_1206_3216Metric, F.Cu at (128.1, 74.0)
- added C64: 100nF, Capacitor_SMD:C_0402_1005Metric, F.Cu at (117.1, 84.0)
- added C65: 10uF, Capacitor_SMD:C_1206_3216Metric, F.Cu at (125.6, 74.0)
- added C66: 100nF, Capacitor_SMD:C_0402_1005Metric, F.Cu at (113.1, 107.1)
- added C67: 10uF, Capacitor_SMD:C_0805_2012Metric, F.Cu at (106.6, 112.5)
- added C68: 10uF, Capacitor_SMD:C_0805_2012Metric, F.Cu at (104.6, 99.5)
- added C69: 10uF, Capacitor_SMD:C_0805_2012Metric, F.Cu at (104.0, 109.0)
- added C70: 10uF, Capacitor_SMD:C_0805_2012Metric, F.Cu at (104.1, 112.5)
- added C71: 10uF, Capacitor_SMD:C_1206_3216Metric, F.Cu at (109.5, 80.1)
- added C72: 100nF, Capacitor_SMD:C_0402_1005Metric, F.Cu at (116.1, 81.5)
- added C73: 10uF, Capacitor_SMD:C_1206_3216Metric, F.Cu at (107.2, 80.1)
- added C74: 10uF, Capacitor_SMD:C_1206_3216Metric, F.Cu at (105.7, 76.3)
- added C75: 47nF, Capacitor_SMD:C_0402_1005Metric, F.Cu at (115.6, 80.0)
- added C76: 47nF, Capacitor_SMD:C_0402_1005Metric, F.Cu at (123.3, 80.2)
- added C77: 47nF, Capacitor_SMD:C_0402_1005Metric, F.Cu at (124.8, 81.2)
- added C78: 4.7uF, Capacitor_SMD:C_0603_1608Metric, F.Cu at (113.6, 81.2)
- added C79: 2.2uF, Capacitor_SMD:C_0805_2012Metric, F.Cu at (108.6, 90.0)
- added C80: 100nF, Capacitor_SMD:C_0402_1005Metric, F.Cu at (118.6, 76.7)
- added C81: 1nF, Capacitor_SMD:C_0402_1005Metric_Pad0.74x0.62mm_HandSolder, F.Cu at (124.6, 78.0)
- added C82: 10uF, Capacitor_SMD:C_1206_3216Metric, F.Cu at (111.1, 73.7)
- added C83: 1nF, Capacitor_SMD:C_0402_1005Metric_Pad0.74x0.62mm_HandSolder, F.Cu at (121.6, 66.2)
- added C84: 10uF, Capacitor_SMD:C_1206_3216Metric, F.Cu at (128.4, 80.0)
- added C85: 10uF, Capacitor_SMD:C_1206_3216Metric, F.Cu at (128.4, 77.5)
- added C86: 10uF, Capacitor_SMD:C_1206_3216Metric, F.Cu at (117.3, 74.0)
- added C87: 10uF, Capacitor_SMD:C_1206_3216Metric, F.Cu at (111.1, 71.2)
- added C88: 10uF, Capacitor_SMD:C_1206_3216Metric, F.Cu at (114.8, 74.0)
- added C89: 100nF, Capacitor_SMD:C_0402_1005Metric, F.Cu at (121.6, 76.7)
- added C90: 10uF, Capacitor_SMD:C_1206_3216Metric, F.Cu at (112.6, 84.0)
- added C91: 100nF, Capacitor_SMD:C_0402_1005Metric, F.Cu at (115.6, 83.0)
- added C92: 10uF, Capacitor_SMD:C_1206_3216Metric, F.Cu at (123.1, 74.0)
- added C93: 22pF, Capacitor_SMD:C_0402_1005Metric, F.Cu at (211.1, 126.2)
- added C94: 1uF, Capacitor_SMD:C_0402_1005Metric, F.Cu at (201.2, 123.3)
- added C95: 47pF, Capacitor_SMD:C_0402_1005Metric, F.Cu at (203.2, 123.3)
- added C96: 10nF, Capacitor_SMD:C_0402_1005Metric_Pad0.74x0.62mm_HandSolder, F.Cu at (215.8, 128.5)
- added C97: 10nF, Capacitor_SMD:C_0402_1005Metric_Pad0.74x0.62mm_HandSolder, F.Cu at (205.2, 123.3)
- added C98: 10uF, Capacitor_SMD:C_0603_1608Metric, F.Cu at (173.9, 45.9)
- added C99: 10uF, Capacitor_SMD:C_0402_1005Metric, F.Cu at (168.2, 70.3)
- added D1: ESDS314DBVR, Package_TO_SOT_SMD:SOT-23-5, F.Cu at (192.0, 57.0)
- added D10: TI ESD501, Package_SON:Texas_DPY0002A_0.6x1mm_P0.65mm, F.Cu at (235.5, 133.2)
- added D11: LED Red, LED_SMD:LED_0805_2012Metric, F.Cu at (235.0, 118.1)
- added D12: LED Blue, LED_SMD:LED_0805_2012Metric, F.Cu at (187.8, 136.0)
- added D13: ESD501, Package_SON:Texas_DPY0002A_0.6x1mm_P0.65mm, F.Cu at (207.1, 117.1)
- added D14: ESD351DPYR, Diode_SMD:D_0402_1005Metric, F.Cu at (168.6, 58.1)
- added D15: RB531SM-30, Diode_SMD:D_SOD-523, F.Cu at (176.1, 62.8)
- added D16: RB531SM-30T2R, Diode_SMD:D_SOD-523, F.Cu at (189.5, 158.2)
- added D17: TPD1E10B06, Package_SON:Texas_DPY0002A_0.6x1mm_P0.65mm, F.Cu at (187.3, 57.0)
- added D18: PGB1010603, Capacitor_SMD:C_0603_1608Metric, F.Cu at (187.4, 43.0)
- added D19: TPD1E10B06, Package_SON:Texas_DPY0002A_0.6x1mm_P0.65mm, F.Cu at (124.5, 46.3)
- added D20: SMF6.0A, Diode_SMD:D_SOD-123F, F.Cu at (223.8, 81.4)
- added D21: BAT54A, Package_TO_SOT_SMD:SOT-23, F.Cu at (228.9, 96.6)
- added D22: BAT54W, Package_TO_SOT_SMD:SOT-323_SC-70, F.Cu at (249.3, 109.5)
- added D9: SS36B, Diode_SMD:D_SMB, F.Cu at (104.1, 86.5)
- added F1: 1A Hold, Fuse:Fuse_0805_2012Metric, F.Cu at (249.5, 98.5)
- added F2: 2A Hold, 4A Trip, Fuse:Fuse_0805_2012Metric, F.Cu at (249.5, 101.4)
- added F3: 1A Hold, Fuse:Fuse_0805_2012Metric, F.Cu at (249.5, 104.3)
- added F4: SMD0805B035TF, Fuse:Fuse_0805_2012Metric, F.Cu at (184.7, 125.7)
- added F5: 10A hold, Fuse:Fuse_2920_7451Metric, F.Cu at (117.1, 111.5)
- added FL1: B39162B4327P810, Filter:Filter_1411-5_1.4x1.1mm, F.Cu at (102.6, 13.4)
- added FL2: 0900LP15B0063001E, easyeda2kicad:FILTER-SMD_0805-8P-L2.0-W1.2-TL, F.Cu at (172.8, 63.2)
- added J10: SOLAR, Connector_JST:JST_PH_S2B-PH-SM4-TB_1x02-1MP_P2.00mm_Horizontal, B.Cu at (151.8, 130.2)
- added J11: Conn_Coaxial, Connector_Coaxial:SMA_Samtec_SMA-J-P-H-ST-EM1_EdgeMount, B.Cu at (151.9, 8.05)
- added J12: Conn_Coaxial_Small, Connector_Coaxial:U.FL_Hirose_U.FL-R-SMT-1_Vertical, F.Cu at (118.3, 7.20)
- added J13: Conn_Coaxial, Connector_Coaxial:SMA_Samtec_SMA-J-P-H-ST-EM1_EdgeMount, F.Cu at (106.8, 8.20)
- added J14: GPIO_Expander, Connector_PinSocket_2.54mm:PinSocket_2x08_P2.54mm_Horizontal, F.Cu at (146.3, 106.9)
- added J8: PD_I2C DEBUG, Connector_PinSocket_2.54mm:PinSocket_1x04_P2.54mm_Vertical, B.Cu at (102.0, 66.3)
- added J9: Conn_01x02, Connector_Molex:Molex_PicoBlade_53261-0271_1x02-1MP_P1.25mm_Horizontal, B.Cu at (156.1, 109.7)
- added JP10: SolderJumper_3_Open, Jumper:SolderJumper-3_P1.3mm_Open_RoundedPad1.0x1.5mm_NumberLabels, F.Cu at (223.1, 132.0)
- added JP11: I2C/UART/SPI, Jumper:SolderJumper-3_P1.3mm_Open_RoundedPad1.0x1.5mm_NumberLabels, F.Cu at (122.8, 18.7)
- added JP12: SolderJumper_3_Bridged12, Jumper:SolderJumper-3_P1.3mm_Bridged12_RoundedPad1.0x1.5mm_NumberLabels, F.Cu at (173.8, 73.5)
- added JP13: DISABLE_GNSS_PROT, Jumper:SolderJumper-2_P1.3mm_Open_RoundedPad1.0x1.5mm, F.Cu at (168.1, 45.9)
- added JP14: BYPASS_FILTER, Resistor_SMD:R_0402_1005Metric, F.Cu at (168.8, 63.6)
- added JP15: ANT_DETECT, Jumper:SolderJumper-2_P1.3mm_Bridged_RoundedPad1.0x1.5mm, F.Cu at (183.8, 158.3)
- added JP16: SolderJumper_3_Bridged12, Jumper:SolderJumper-3_P1.3mm_Bridged12_RoundedPad1.0x1.5mm_NumberLabels, F.Cu at (181.8, 136.5)
- added JP17: DISABLE_5V_PROT, Jumper:SolderJumper-2_P1.3mm_Open_RoundedPad1.0x1.5mm, F.Cu at (188.6, 131.0)
- added JP4: I2C_SDA_PULLUP, Jumper:SolderJumper-2_P1.3mm_Bridged_RoundedPad1.0x1.5mm, F.Cu at (210.6, 32.1)
- added JP6: WRITE_PROTECT, Jumper:SolderJumper-3_P1.3mm_Bridged12_RoundedPad1.0x1.5mm_NumberLabels, F.Cu at (243.9, 79.7)
- added JP7: ZVC, Jumper:SolderJumper-2_P1.3mm_Open_RoundedPad1.0x1.5mm, F.Cu at (111.1, 107.9)
- added JP8: TIMEPULSE, Jumper:SolderJumper-2_P1.3mm_Bridged_RoundedPad1.0x1.5mm, F.Cu at (232.0, 117.8)
- added JP9: TIMEPULSE, Jumper:SolderJumper-2_P1.3mm_Bridged_RoundedPad1.0x1.5mm, F.Cu at (219.6, 132.0)
- added L3: 470nH, Inductor_SMD:L_0603_1608Metric, F.Cu at (168.6, 60.6)
- added L4: 2.2uH, Inductor_SMD:L_Sunlord_MWSA1003S, F.Cu at (151.8, 68.5)
- added L5: 3.3uH 11A Sat, Inductor_SMD:L_APV_APH1040, F.Cu at (151.8, 80.0)
- added NT1: NetTie_3, NetTie:NetTie-3_SMD_Pad0.5mm, F.Cu at (212.9, 42.5)
- added NT2: NetTie_3, NetTie:NetTie-3_SMD_Pad0.5mm, F.Cu at (212.9, 44.0)
- added Q10: SI2308, Package_TO_SOT_SMD:SOT-23, F.Cu at (109.3, 85.9)
- added Q11: CSD17581Q3A, Package_SON:VSON-8_3.3x3.3mm_P0.65mm_NexFET, F.Cu at (129.3, 83.1)
- added Q12: AO3401A, Package_TO_SOT_SMD:SOT-23, F.Cu at (196.2, 68.2)
- added Q13: BSS138, Package_TO_SOT_SMD:SOT-23, F.Cu at (194.9, 79.3)
- added Q14: 2N7002, Package_TO_SOT_SMD:SOT-23, F.Cu at (222.1, 71.9)
- added Q15: 2N7002, Package_TO_SOT_SMD:SOT-23, F.Cu at (222.1, 76.4)
- added Q2: CSD15380F3, Package_DFN_QFN:Texas_PicoStar_DFN-3_0.69x0.60mm, F.Cu at (185.2, 65.4)
- added Q5: AON7534, easyeda2kicad:PQFN-8_L3.1-W3.1-P0.65-LS3.3-BL, F.Cu at (104.6, 105.6)
- added Q6: AON7534, easyeda2kicad:PQFN-8_L3.1-W3.1-P0.65-LS3.3-BL, F.Cu at (104.6, 102.3)
- added Q7: CSD18512Q5B, Package_SON:VSONP-8-1EP_5x6_P1.27mm, F.Cu at (114.7, 91.2)
- added Q8: CSD18512Q5B, Package_SON:VSONP-8-1EP_5x6_P1.27mm, F.Cu at (120.2, 91.2)
- added Q9: SI2308, Package_TO_SOT_SMD:SOT-23, F.Cu at (104.3, 80.6)
- added R100: 0, Resistor_SMD:R_0805_2012Metric, F.Cu at (197.3, 146.9)
- added R101: 10k, Resistor_SMD:R_0402_1005Metric, F.Cu at (197.3, 148.9)
- added R102: 1M, Resistor_SMD:R_0402_1005Metric, F.Cu at (191.0, 150.2)
- added R103: 100, Resistor_SMD:R_0402_1005Metric, F.Cu at (189.0, 161.3)
- added R104: 402k, Resistor_SMD:R_0603_1608Metric, F.Cu at (179.3, 154.9)
- added R105: 100k, Resistor_SMD:R_0402_1005Metric, F.Cu at (179.3, 156.9)
- added R106: 100k, Resistor_SMD:R_0402_1005Metric, F.Cu at (197.3, 150.9)
- added R107: 402k, Resistor_SMD:R_0603_1608Metric, F.Cu at (197.3, 152.9)
- added R108: 100k, Resistor_SMD:R_0402_1005Metric, F.Cu at (200.2, 145.0)
- added R109: 6.04k, Resistor_SMD:R_0402_1005Metric_Pad0.72x0.64mm_HandSolder, F.Cu at (179.3, 158.9)
- added R110: 6.04k, Resistor_SMD:R_0402_1005Metric_Pad0.72x0.64mm_HandSolder, F.Cu at (191.0, 152.8)
- added R111: 100, Resistor_SMD:R_0402_1005Metric_Pad0.72x0.64mm_HandSolder, F.Cu at (200.2, 146.9)
- added R112: 2.2, Resistor_SMD:R_0805_2012Metric, F.Cu at (200.2, 148.9)
- added R113: 10k, Resistor_SMD:R_0402_1005Metric, F.Cu at (204.0, 33.3)
- added R114: 10, Resistor_SMD:R_0402_1005Metric, F.Cu at (204.0, 35.3)
- added R115: 402k, Resistor_SMD:R_0603_1608Metric, F.Cu at (193.0, 74.3)
- added R116: 174k, Resistor_SMD:R_0402_1005Metric_Pad0.72x0.64mm_HandSolder, F.Cu at (204.0, 37.3)
- added R117: 100, Resistor_SMD:R_0402_1005Metric_Pad0.72x0.64mm_HandSolder, F.Cu at (197.3, 56.1)
- added R118: 2.2, Resistor_SMD:R_0805_2012Metric, F.Cu at (206.9, 31.3)
- added R119: 10k, Resistor_SMD:R_0402_1005Metric, F.Cu at (200.2, 150.9)
- added R120: 10, Resistor_SMD:R_0402_1005Metric, F.Cu at (206.9, 33.3)
- added R121: 402k, Resistor_SMD:R_0603_1608Metric, F.Cu at (195.4, 56.1)
- added R122: 101k, Resistor_SMD:R_0805_2012Metric_Pad1.20x1.40mm_HandSolder, F.Cu at (206.9, 35.3)
- added R123: 1k, Resistor_SMD:R_0402_1005Metric_Pad0.72x0.64mm_HandSolder, F.Cu at (171.0, 53.8)
- added R124: 1k, Resistor_SMD:R_0402_1005Metric_Pad0.72x0.64mm_HandSolder, F.Cu at (205.3, 59.4)
- added R125: 86.6k, Resistor_SMD:R_0402_1005Metric, F.Cu at (203.3, 59.4)
- added R126: 3.92k, Resistor_SMD:R_0402_1005Metric, F.Cu at (201.3, 59.4)
- added R127: 27.4k, Resistor_SMD:R_0402_1005Metric, F.Cu at (199.3, 59.4)
- added R128: 750, Resistor_SMD:R_0402_1005Metric_Pad0.72x0.64mm_HandSolder, F.Cu at (197.3, 59.4)
- added R129: 280k, Resistor_SMD:R_0603_1608Metric, F.Cu at (206.9, 37.3)
- added R130: 100k, Resistor_SMD:R_0402_1005Metric, F.Cu at (195.4, 59.4)
- added R131: 100k, Resistor_SMD:R_0402_1005Metric, F.Cu at (226.0, 72.7)
- added R132: 10k, Resistor_SMD:R_0402_1005Metric, F.Cu at (226.0, 74.7)
- added R133: 10k, Resistor_SMD:R_0402_1005Metric_Pad0.72x0.64mm_HandSolder, F.Cu at (92.9, 95.7)
- added R30: 100k, Resistor_SMD:R_0402_1005Metric, F.Cu at (234.7, 75.2)
- added R31: 1M, Resistor_SMD:R_0402_1005Metric, F.Cu at (225.6, 92.2)
- added R32: 0, Resistor_SMD:R_0402_1005Metric, F.Cu at (234.7, 77.2)
- added R33: 0, Resistor_SMD:R_0402_1005Metric, F.Cu at (228.1, 106.5)
- added R34: 0, Resistor_SMD:R_0402_1005Metric, F.Cu at (232.1, 110.2)
- added R35: 10k, Resistor_SMD:R_0402_1005Metric, F.Cu at (201.1, 31.3)
- added R36: 2.2k, Resistor_SMD:R_0402_1005Metric, F.Cu at (193.1, 61.8)
- added R37: 2.2k, Resistor_SMD:R_0402_1005Metric, F.Cu at (190.6, 61.8)
- added R38: 10k, Resistor_SMD:R_0402_1005Metric, F.Cu at (188.1, 61.8)
- added R39: 150, Resistor_SMD:R_1206_3216Metric, F.Cu at (112.2, 97.3)
- added R40: 150, Resistor_SMD:R_1206_3216Metric, F.Cu at (121.8, 100.8)
- added R41: 5m, Resistor_SMD:R_0805_2012Metric_Pad1.20x1.40mm_HandSolder, F.Cu at (121.6, 103.0)
- added R42: 10, Resistor_SMD:R_0402_1005Metric, F.Cu at (109.3, 101.0)
- added R43: 1k, Resistor_SMD:R_0402_1005Metric, F.Cu at (115.7, 107.0)
- added R44: 100, Resistor_SMD:R_0402_1005Metric, F.Cu at (109.1, 102.8)
- added R45: 1k, Resistor_SMD:R_0402_1005Metric, F.Cu at (111.8, 105.3)
- added R46: 10k, Resistor_SMD:R_0402_1005Metric, F.Cu at (116.7, 107.0)
- added R47: 330, Resistor_SMD:R_1210_3225Metric, F.Cu at (107.5, 109.0)
- added R48: 100, Resistor_SMD:R_0402_1005Metric, F.Cu at (110.6, 104.0)
- added R49: 2, Resistor_SMD:R_0402_1005Metric, F.Cu at (113.8, 86.7)
- added R50: 10k, Resistor_SMD:R_0402_1005Metric, F.Cu at (114.0, 107.0)
- added R51: 5.24k, Resistor_SMD:R_0603_1608Metric_Pad0.98x0.95mm_HandSolder, F.Cu at (122.8, 86.0)
- added R52: 30.31k, Resistor_SMD:R_0603_1608Metric_Pad0.98x0.95mm_HandSolder, F.Cu at (124.3, 88.0)
- added R53: 294, Resistor_SMD:R_0402_1005Metric, F.Cu at (119.3, 85.0)
- added R54: 24.3k, Resistor_SMD:R_0603_1608Metric_Pad0.98x0.95mm_HandSolder, F.Cu at (128.1, 87.0)
- added R55: 68.1k, Resistor_SMD:R_0603_1608Metric_Pad0.98x0.95mm_HandSolder, F.Cu at (124.3, 83.5)
- added R56: 100k, Resistor_SMD:R_0402_1005Metric, F.Cu at (121.3, 85.0)
- added R57: 294, Resistor_SMD:R_0402_1005Metric, F.Cu at (118.3, 85.0)
- added R58: 8.2k, Resistor_SMD:R_0402_1005Metric_Pad0.72x0.64mm_HandSolder, F.Cu at (124.8, 82.2)
- added R59: 100, Resistor_SMD:R_0402_1005Metric, F.Cu at (120.3, 85.0)
- added R60: 294, Resistor_SMD:R_0402_1005Metric, F.Cu at (102.1, 81.5)
- added R61: 294, Resistor_SMD:R_0402_1005Metric, F.Cu at (107.3, 83.2)
- added R62: 2, Resistor_SMD:R_0402_1005Metric, F.Cu at (107.1, 89.5)
- added R63: 100, Resistor_SMD:R_0402_1005Metric, F.Cu at (127.3, 85.5)
- added R64: 2.2, Resistor_SMD:R_0402_1005Metric_Pad0.72x0.64mm_HandSolder, F.Cu at (123.6, 78.0)
- added R65: 2.2, Resistor_SMD:R_0402_1005Metric_Pad0.72x0.64mm_HandSolder, F.Cu at (119.3, 66.2)
- added R66: 3k, Resistor_SMD:R_0402_1005Metric_Pad0.72x0.64mm_HandSolder, F.Cu at (112.3, 76.8)
- added R67: 10k, Resistor_SMD:R_0402_1005Metric, F.Cu at (229.2, 138.6)
- added R68: 2.2k, Resistor_SMD:R_0402_1005Metric_Pad0.72x0.64mm_HandSolder, F.Cu at (230.5, 127.0)
- added R69: 0, Resistor_SMD:R_0402_1005Metric, F.Cu at (233.0, 127.0)
- added R70: 2k, Resistor_SMD:R_0402_1005Metric, F.Cu at (235.5, 127.0)
- added R71: 1k, Resistor_SMD:R_0402_1005Metric, F.Cu at (231.2, 138.6)
- added R72: 2.2k, Resistor_SMD:R_0402_1005Metric_Pad0.72x0.64mm_HandSolder, F.Cu at (233.2, 138.6)
- added R73: 0, Resistor_SMD:R_0402_1005Metric, F.Cu at (168.1, 47.9)
- added R74: 62, Resistor_SMD:R_0805_2012Metric, F.Cu at (168.1, 49.8)
- added R75: 0, Resistor_SMD:R_0402_1005Metric_Pad0.72x0.64mm_HandSolder, F.Cu at (168.1, 51.8)
- added R76: 10k, Resistor_SMD:R_0402_1005Metric, F.Cu at (168.2, 66.4)
- added R77: 100k, Resistor_SMD:R_0402_1005Metric, F.Cu at (168.1, 53.8)
- added R78: 1k, Resistor_SMD:R_0402_1005Metric, F.Cu at (168.1, 55.8)
- added R79: 100k, Resistor_SMD:R_0402_1005Metric, F.Cu at (171.0, 45.9)
- added R80: 150, Resistor_SMD:R_0402_1005Metric_Pad0.72x0.64mm_HandSolder, F.Cu at (177.7, 58.3)
- added R81: 37.4, Resistor_SMD:R_0402_1005Metric_Pad0.72x0.64mm_HandSolder, F.Cu at (226.0, 70.7)
- added R82: 4.7k, Resistor_SMD:R_0402_1005Metric, F.Cu at (171.0, 49.8)
- added R83: 150, Resistor_SMD:R_0402_1005Metric_Pad0.72x0.64mm_HandSolder, F.Cu at (171.0, 51.8)
- added R84: 150k, Resistor_SMD:R_0402_1005Metric, F.Cu at (194.4, 145.0)
- added R85: 215k, Resistor_SMD:R_0603_1608Metric_Pad0.98x0.95mm_HandSolder, F.Cu at (187.0, 155.3)
- added R86: 100k, Resistor_SMD:R_0402_1005Metric, F.Cu at (194.4, 146.9)
- added R87: 113k, Resistor_SMD:R_0603_1608Metric_Pad0.98x0.95mm_HandSolder, F.Cu at (194.4, 148.9)
- added R88: 6.65k, Resistor_SMD:R_0603_1608Metric_Pad0.98x0.95mm_HandSolder, F.Cu at (191.0, 145.2)
- added R89: 200k, Resistor_SMD:R_0603_1608Metric_Pad0.98x0.95mm_HandSolder, F.Cu at (194.4, 150.9)
- added R90: 301k, Resistor_SMD:R_0402_1005Metric, F.Cu at (179.3, 145.0)
- added R91: 100k, Resistor_SMD:R_0402_1005Metric, F.Cu at (179.3, 146.9)
- added R92: 10k, Resistor_SMD:R_0402_1005Metric, F.Cu at (179.3, 148.9)
- added R93: 0, Resistor_SMD:R_0402_1005Metric, F.Cu at (175.2, 157.6)
- added R94: 10k, Resistor_SMD:R_0402_1005Metric, F.Cu at (194.4, 152.9)
- added R95: 0, Resistor_SMD:R_0402_1005Metric_Pad0.72x0.64mm_HandSolder, F.Cu at (197.3, 145.0)
- added R96: 100k, Resistor_SMD:R_0402_1005Metric, F.Cu at (191.0, 147.7)
- added R97: 10k, Resistor_SMD:R_0402_1005Metric, F.Cu at (179.3, 150.9)
- added R98: 22, Resistor_SMD:R_0402_1005Metric, F.Cu at (179.3, 152.9)
- added R99: 1k, Resistor_SMD:R_0402_1005Metric, F.Cu at (175.2, 160.6)
- added RN1: 10k, Resistor_SMD:R_Array_Concave_4x0402, F.Cu at (253.3, 101.3)
- added SW2: BOOT, Button_Switch_SMD:SW_Push_SPST_NO_Alps_SKRK, F.Cu at (111.8, 132.9)
- added SW3: POWER/RESET, Button_Switch_SMD:SW_Push_SPST_NO_Alps_SKRK, F.Cu at (126.8, 91.2)
- added SW4: RESET_GNSS, Button_Switch_SMD:SW_Push_SPST_NO_Alps_SKRK, F.Cu at (103.1, 23.9)
- added SW5: SAFEBOOT_GNSS, Button_Switch_SMD:SW_Push_SPST_NO_Alps_SKRK, F.Cu at (124.1, 8.45)
- added TH1: 103AT 10k, Resistor_SMD:R_0603_1608Metric, B.Cu at (142.3, 28.4)
- added TH2: 103AT 10k, Resistor_SMD:R_0603_1608Metric, B.Cu at (118.4, 28.7)
- added TH3: 103AT 10k, Resistor_SMD:R_0603_1608Metric, B.Cu at (141.8, 77.5)
- added TH4: 103AT 10k, Resistor_SMD:R_0603_1608Metric, B.Cu at (142.2, 55.9)
- added TH5: 103AT 10k, Resistor_SMD:R_0603_1608Metric, B.Cu at (116.5, 76.3)
- added TP10: PGOOD, TestPoint:TestPoint_Loop_D2.54mm_Drill1.5mm_Beaded, F.Cu at (174.7, 146.8)
- added TP11: PGOOD, TestPoint:TestPoint_Loop_D2.54mm_Drill1.5mm_Beaded, F.Cu at (174.7, 151.9)
- added TP12: 3V3, TestPoint:TestPoint_2Pads_Pitch2.54mm_Drill0.8mm, F.Cu at (194.7, 129.2)
- added TP13: 5V_RAW, TestPoint:TestPoint_2Pads_Pitch2.54mm_Drill0.8mm, F.Cu at (194.7, 132.6)
- added TP14: 5V, TestPoint:TestPoint_2Pads_Pitch2.54mm_Drill0.8mm, F.Cu at (194.7, 135.9)
- added TP2: IN_CP, TestPoint:TestPoint_2Pads_Pitch2.54mm_Drill0.8mm, F.Cu at (105.8, 97.0)
- added TP3: REG3, TestPoint:TestPoint_Pad_D1.5mm, F.Cu at (120.3, 105.5)
- added TP4: PPHV, TestPoint:TestPoint_2Pads_Pitch2.54mm_Drill0.8mm, F.Cu at (102.8, 91.5)
- added TP5: CS_GPS, TestPoint:TestPoint_Loop_D1.80mm_Drill1.0mm_Beaded, F.Cu at (220.1, 120.3)
- added TP6: 5V_LORA, TestPoint:TestPoint_2Pads_Pitch2.54mm_Drill0.8mm, F.Cu at (177.1, 53.2)
- added TP7: EN_3V3, TestPoint:TestPoint_Pad_D1.5mm, F.Cu at (181.4, 140.1)
- added TP8: VSYS, TestPoint:TestPoint_2Pads_Pitch2.54mm_Drill0.8mm, F.Cu at (194.7, 122.5)
- added TP9: VSYS, TestPoint:TestPoint_2Pads_Pitch2.54mm_Drill0.8mm, F.Cu at (194.7, 125.9)
- added U10: TPS7A2033PDBVR, easyeda2kicad:SOT-23-5_L2.9-W1.6-P0.95-LS2.8-BR, F.Cu at (107.6, 45.7)
- added U11: TPS259474LRPWR, easyeda2kicad:VQFN-10_L2.0-W2.0-P0.45-TL, F.Cu at (111.2, 45.4)
- added U12: E22P-915M30S, footprints:COMM-SMD_22P-P2.54-L38.5-W24.0_E22-400M33S, F.Cu at (137.0, 32.3)
- added U13: LM61460AASQRJRRQ1, easyeda2kicad:VQFN-14-HR_L4.0-W3.5-TL_LM61460AASQRJRRQ1, F.Cu at (169.9, 159.6)
- added U14: LM61460AASQRJRRQ1, easyeda2kicad:VQFN-14-HR_L4.0-W3.5-TL_LM61460AASQRJRRQ1, F.Cu at (195.3, 139.6)
- added U15: TPS259474ARPWR, easyeda2kicad:VQFN-10_L2.0-W2.0-P0.45-TL, F.Cu at (179.2, 161.4)
- added U16: SN74LVC1G74, Package_SON:X2SON-8_1.4x1mm_P0.35mm, F.Cu at (194.9, 42.9)
- added U17: TCAL9539RTWR_C22445413, easyeda2kicad:TQFN-24_L4.0-W4.0-P0.50-BL-EP2.3, F.Cu at (94.1, 89.0)
- added U5: TI TPS25751DREFR, Package_DFN_QFN:Texas_REF0038A_WQFN-38-2EP_6x4mm_P0.4, F.Cu at (142.9, 116.8)
- added U8: BQ25798, Package_DFN_QFN:Texas_RQM0029A_VQFN-29_4x4mm_P0.4mm, F.Cu at (120.1, 81.0)
- added U9: NEO-M9N, RF_GPS:ublox_NEO, F.Cu at (113.3, 25.4)
- added Y1: 32.768KHz, Crystal:Crystal_SMD_3215-2Pin_3.2x1.5mm, F.Cu at (187.8, 39.9)
- added Y2: SX1M4.000M10F30TNN, Oscillator:Oscillator_SMD_SiT_PQFN-4Pin_2.0x1.6mm, F.Cu at (199.3, 139.4)
- BT1: value Battery_Cell -> 21700 Li-ion; footprint Battery:BatteryHolder_Keystone_1042_1x18650 -> easyeda2kicad:BAT-SMD_L82.5.5-W25-BH-21700-B1BJ001
- C1, C13, C15, C2, C3, C8: value 10uF -> 2.2uF
- C10: value 100nF 16V -> 10uF; footprint Capacitor_SMD:C_0402_1005Metric -> Capacitor_SMD:C_0603_1608Metric
- C11: value 100nF -> 10uF; footprint Capacitor_SMD:C_0402_1005Metric -> Capacitor_SMD:C_0603_1608Metric
- C12, C25: value 100nF -> 1uF
- C14: value 47uF -> 10uF
- C16, C24, C5, C9: value 10uF -> 100nF
- C17, C20: value 10uF -> 1uF
- C18: value 47uF -> 1uF; footprint Capacitor_SMD:C_0805_2012Metric -> Capacitor_SMD:C_0402_1005Metric
- C21: value 100nF -> 10nF
- C22, C23: value 10uF -> 10nF
- C26: value 680uF -> 10uF; footprint Capacitor_SMD:CP_Elec_8x10 -> Capacitor_SMD:C_1206_3216Metric
- C27: footprint Capacitor_SMD:C_0402_1005Metric -> Capacitor_SMD:C_1206_3216Metric
- C6, C7: value 10uF -> 7pF
- D2: value LED Red -> ESDS314DBVR; footprint LED_THT:LED_D5.0mm -> Package_TO_SOT_SMD:SOT-23-5
- D3: value LED Blue -> ESDS314DBVR; footprint LED_THT:LED_D5.0mm -> Package_TO_SOT_SMD:SOT-23-5
- D4: value ESDS314DBVR-TP -> 1N5819WS; footprint Package_TO_SOT_SMD:SOT-23-5 -> Diode_SMD:D_SOD-323
- D5: value ESDS314DBVR-TP -> SMF10A; footprint Package_TO_SOT_SMD:SOT-23-5 -> Diode_SMD:D_SOD-123; moved to B.Cu
- D6: value SMAJ3.3A -> BAV199; footprint Diode_SMD:D_SMA-SMB_Universal_Handsoldering -> Package_TO_SOT_SMD:SOT-23
- D7: value BESDU0603-14 -> SMF24A; footprint Diode_SMD:D_0603_1608Metric -> Diode_SMD:D_SOD-123F
- D8: value BESDU0603-14 -> CHARGING; footprint Diode_SMD:D_0603_1608Metric -> LED_SMD:LED_0805_2012Metric
- FB1: value FerriteBead -> BLM18HG601SN1D
- J1: value I2C1 -> SPI BUS; footprint Connector_PinSocket_2.54mm:PinSocket_1x04_P2.54mm_Horizontal -> Connector_PinSocket_2.54mm:PinSocket_1x06_P2.54mm_Horizontal; moved to B.Cu
- J2: value SPI BUS -> I2C3; footprint Connector_PinSocket_2.54mm:PinSocket_1x06_P2.54mm_Horizontal -> Connector_JST:JST_SH_SM04B-SRSS-TB_1x04-1MP_P1.00mm_Horizontal; moved to B.Cu
- J3: value Conn_Coaxial -> I2C1; footprint Connector_Coaxial:SMA_Samtec_SMA-J-P-H-ST-EM1_EdgeMount -> Connector_PinSocket_2.54mm:PinSocket_1x04_P2.54mm_Horizontal; moved to B.Cu
- J4: value Conn_Coaxial_Small -> I2C2; footprint Connector_Coaxial:U.FL_Hirose_U.FL-R-SMT-1_Vertical -> Connector_PinSocket_2.54mm:PinSocket_1x04_P2.54mm_Vertical; moved to B.Cu
- J5: value Conn_Coaxial -> e-Ink Display Connector; footprint Connector_Coaxial:SMA_Samtec_SMA-J-P-H-ST-EM1_EdgeMount -> Connector_Molex:Molex_PicoBlade_53261-0871_1x08-1MP_P1.25mm_Horizontal; moved to B.Cu
- J6: value Conn_01x02 -> UART0; footprint Connector_Molex:Molex_PicoBlade_53261-0271_1x02-1MP_P1.25mm_Horizontal -> Connector_JST:JST_SH_SM03B-SRSS-TB_1x03-1MP_P1.00mm_Horizontal; moved to B.Cu
- J7: value I2C2 -> GCT USB4105-GF-A-120; footprint Connector_PinSocket_2.54mm:PinSocket_1x04_P2.54mm_Vertical -> Connector_USB:USB_C_Receptacle_GCT_USB4105-xx-A_16P_TopMnt_Horizontal; moved to F.Cu
- JP1, JP2: value TIMEPULSE -> SolderJumper_2_Open; footprint Jumper:SolderJumper-2_P1.3mm_Bridged_RoundedPad1.0x1.5mm -> Jumper:SolderJumper-2_P1.3mm_Open_TrianglePad1.0x1.5mm
- JP3: value SolderJumper_3_Open -> I2C_IRQ_PULLUP; footprint Jumper:SolderJumper-3_P1.3mm_Open_RoundedPad1.0x1.5mm_NumberLabels -> Jumper:SolderJumper-2_P1.3mm_Bridged_RoundedPad1.0x1.5mm
- JP5: value SolderJumper_3_Open -> I2C_SCL_PULLUP; footprint Jumper:SolderJumper-3_P1.3mm_Open_RoundedPad1.0x1.5mm_NumberLabels -> Jumper:SolderJumper-2_P1.3mm_Bridged_RoundedPad1.0x1.5mm
- L1: value 22nH -> 2.2uH; footprint Inductor_SMD:L_0603_1608Metric -> Inductor_SMD:L_Vishay_IFSC-1515AH_4x4x1.8mm
- L2: value 470nH -> 47nH; footprint Inductor_SMD:L_1008_2520Metric_Pad1.43x2.20mm_HandSolder -> Inductor_SMD:L_0603_1608Metric
- Q1: value AO3401A -> CSD25480F3; footprint Package_TO_SOT_SMD:SOT-23 -> Package_DFN_QFN:Texas_PicoStar_DFN-3_0.69x0.60mm
- Q3: value CSD16301Q2 -> CSD25480F3; footprint Package_SON:Texas_DQK -> Package_DFN_QFN:Texas_PicoStar_DFN-3_0.69x0.60mm
- Q4: value CSD16301Q2 -> CSD15380F3; footprint Package_SON:Texas_DQK -> Package_DFN_QFN:Texas_PicoStar_DFN-3_0.69x0.60mm
- R1, R2: value 4.7k -> 33; footprint Resistor_SMD:R_0402_1005Metric -> Resistor_SMD:R_0402_1005Metric_Pad0.72x0.64mm_HandSolder
- R10, R11: value 2k -> 22; footprint Resistor_SMD:R_0402_1005Metric -> Resistor_SMD:R_0402_1005Metric_Pad0.72x0.64mm_HandSolder
- R12: value 2.2k -> 0; footprint Resistor_SMD:R_0603_1608Metric -> Resistor_SMD:R_0402_1005Metric
- R13: value 10 -> 0
- R14, R5, R6: value 22 -> 0
- R15, R18: value 10k -> 0
- R17: value 10k -> 22
- R19: value 2.2k -> 0
- R20: value 330 -> 10k; footprint Resistor_SMD:R_0402_1005Metric -> Resistor_SMD:R_0402_1005Metric_Pad0.72x0.64mm_HandSolder
- R21: value 100 -> 2.2k; footprint Resistor_SMD:R_0402_1005Metric -> Resistor_SMD:R_0402_1005Metric_Pad0.72x0.64mm_HandSolder
- R22: value 1k -> 2.2k; footprint Resistor_SMD:R_0402_1005Metric -> Resistor_SMD:R_0402_1005Metric_Pad0.72x0.64mm_HandSolder
- R23: value 2M -> 100k; footprint Resistor_SMD:R_0402_1005Metric -> Resistor_SMD:R_0402_1005Metric_Pad0.72x0.64mm_HandSolder
- R24: value 680k -> 10k; footprint Resistor_SMD:R_0402_1005Metric -> Resistor_SMD:R_0402_1005Metric_Pad0.72x0.64mm_HandSolder
- R25, R26: value 100k -> 10k; footprint Resistor_SMD:R_0402_1005Metric -> Resistor_SMD:R_0402_1005Metric_Pad0.72x0.64mm_HandSolder
- R27, R28: value 0 -> 100k; footprint Resistor_SMD:R_0603_1608Metric -> Resistor_SMD:R_0402_1005Metric
- R29: value 0 -> 1M
- R3, R4: value 22 -> 33; footprint Resistor_SMD:R_0402_1005Metric -> Resistor_SMD:R_0402_1005Metric_Pad0.72x0.64mm_HandSolder
- R8: value 10k -> 10M; footprint Resistor_SMD:R_0402_1005Metric -> Resistor_SMD:R_0805_2012Metric
- R9: value 2.2k -> 10k; footprint Resistor_SMD:R_0603_1608Metric -> Resistor_SMD:R_0402_1005Metric
- SW1: value SW_Push -> ESP_RESET
- TP1: value TestPoint_Probe -> R_SENSE_SHUNT; footprint TestPoint:TestPoint_Loop_D1.80mm_Drill1.0mm_Beaded -> TestPoint:TestPoint_2Pads_Pitch2.54mm_Drill0.8mm
- U1: value XIAO-ESP32-C6-SMD -> ESP32-S3-WROOM-1; footprint footprints:XIAO-ESP32-C6-SMD -> RF_Module:ESP32-S3-WROOM-1
- U2: value NEO-M9N -> QMC6309; footprint RF_GPS:ublox_NEO -> easyeda2kicad:X1-WLB0808-4_L0.8-W0.8-P0.40-TL
- U3: value E22P-915M30S -> TVS2200DRV; footprint footprints:COMM-SMD_22P-P2.54-L38.5-W24.0_E22-400M33S -> Package_SON:WSON-6-1EP_2x2mm_P0.65mm_EP1x1.6mm
- U4: value BQ29700 -> TPD8S300/A; footprint Package_SON:WSON-6_1.5x1.5mm_P0.5mm -> easyeda2kicad:WQFN-20_L3.0-W3.0-P0.40-TL-EP1.7
- U6: value TPS2116DRL -> CAT24C256; footprint Package_TO_SOT_SMD:SOT-583-8 -> Package_DFN_QFN:OnSemi_UDFN-8_1.2x1.8mm_P0.4mm
- U7: value TPS61033DRLR -> MAX17320G22+; footprint Package_TO_SOT_SMD:SOT-583-8 -> easyeda2kicad:QFN-24_L4.0-W4.0-P0.50-BL-EP2.6
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Connections:
- BT1 pad 2: -BATT -> Net-(BT1--)
- C10 pad 1: Net-(C10-Pad1) -> +3V3
- C11 pad 1: /NRST_LORA -> +3V3
- C12 pad 1: +5V -> +3V3
- C13 pad 1: +5V -> Net-(J5-Pin_8)
- C14 pad 1: +5V -> Net-(J5-Pin_8)
- C15 pad 1: +5V -> GND
- C15 pad 2: GND -> +3V3
- C16 pad 1: +3V3 -> GND
- C16 pad 2: GND -> +3V3
- C18 pad 1: +5V -> GND
- C18 pad 2: GND -> PD_LDO_3V3
- C19 pad 1: -BATT -> Net-(U4-VBIAS)
- C19 pad 2: Net-(U4-BAT) -> GND
- C20 pad 1: Net-(BT1-+) -> PD_LDO_3V3
- C20 pad 2: -BATT -> GND
- C21 pad 1: Net-(U7-EN) -> VBUS
- C22 pad 1: Net-(U7-EN) -> VBUS
- C23 pad 1: Net-(U7-VOUT) -> VBUS
- C24 pad 1: Net-(U7-VOUT) -> VBUS
- C25 pad 2: Net-(U1-GPIO0_A0_D0) -> PD_LDO_3V3
- C26 pad 1: +5V -> PPHV
- C27 pad 1: +3V3 -> PPHV
- C4 pad 2: +3V3 -> Net-(C4-Pad2)
- C5 pad 1: VBUS -> GND
- C5 pad 2: GND -> Net-(C5-Pad2)
- C6 pad 1: VBUS -> GND
- C6 pad 2: GND -> Net-(C6-Pad2)
- C7 pad 1: VBUS -> GND
- C7 pad 2: GND -> Net-(C7-Pad2)
- C9 pad 1: +3V3 -> GND
- C9 pad 2: GND -> /Root/EN
- D2 pad 1: GND -> I2C_HOST_SCL
- D2 pad 2: Net-(D2-A) -> GND
- D3 pad 1: GND -> /Root/D/C_DISPLAY
- D3 pad 2: Net-(D3-A) -> GND
- D4 pad 1: /SCL_I2C -> Net-(D4-K)
- D4 pad 2: GND -> +3V3
- D5 pad 1: /SCK -> Net-(BT1-+)
- D5 pad 2: GND -> -BATT
- D6 pad 1: +3V3 -> -BATT
- D6 pad 2: GND -> Net-(D6-common)
- D7 pad 1: GND -> SOLAR
- D7 pad 2: GPS_ANT -> GND
- D8 pad 1: GND -> Net-(D8-K)
- D8 pad 2: /LORA/LORA_ANT -> Net-(D8-A)
- FB1 pad 1: +5V -> Net-(Q12-S)
- FB1 pad 2: Net-(U7-VOUT) -> Net-(JP12-C)
- J1 pad 1: +3V3 -> Net-(J1-Pin_1)
- J1 pad 3: /SCL_I2C -> Net-(J1-Pin_3)
- J1 pad 4: /SDA_I2C -> Net-(J1-Pin_4)
- J2 pad 1: +3V3 -> GND
- J2 pad 2: GND -> +3V3
- J2 pad 3: /SCK -> I2C_HOST_SCL
- J2 pad 4: /MOSI -> I2C_HOST_SDA
- J3 pad 1: /GNSS/AFT_GPS_ANT -> Net-(J3-Pin_1)
- J4 pad 1: Net-(J4-In) -> Net-(J4-Pin_1)
- J5 pad 1: /LORA/LORA_ANT -> /Root/BUSY_DISPLAY
- J5 pad 2: GND -> /Root/RESET_DISPLAY
- J6 pad 1: -BATT -> GND
- J6 pad 2: Net-(BT1-+) -> Net-(J6-Pin_2)
- J6 pad MP: unconnected-(J6-MountPin-PadMP)_1 -> (no net)
- JP1 pad 1: +3V3 -> I2C_HOST_SDA
- JP1 pad 2: Net-(JP1-B) -> /Root/GNSS/SDA/SPI_CS
- JP2 pad 1: /GNSS/PPS -> I2C_HOST_SCL
- JP2 pad 2: Net-(JP2-B) -> /Root/GNSS/SCL/SPI_CLK
- JP3 pad 1: Net-(JP3-A) -> I2C_HOST_IRQ
- JP3 pad 2: +3V3 -> Net-(JP3-B)
- JP5 pad 1: GND -> I2C_HOST_SCL
- JP5 pad 2: /GNSS/D_SEL -> Net-(JP5-B)
- L1 pad 1: GPS_ANT -> Net-(U8-SW1)
- L1 pad 2: Net-(C10-Pad1) -> Net-(U8-SW2)
- L2 pad 1: Net-(U7-EN) -> Net-(C95-Pad2)
- L2 pad 2: Net-(U7-SW) -> Net-(C93-Pad1)
- Q1 pad 1: Net-(Q1-G) -> /USB Interface/GPIO2
- Q1 pad 2: +BATT -> PD_LDO_3V3
- Q1 pad 3: Net-(BT1-+) -> Net-(Q1-D)
- Q3 pad 1: Net-(Q3-D-Pad1) -> /USB Interface/GPIO2
- Q3 pad 2: Net-(Q3-D-Pad1) -> PD_LDO_3V3
- Q3 pad 3: Net-(Q3-G) -> Net-(Q3-D)
- Q4 pad 1: Net-(Q3-D-Pad1) -> /USB Interface/GPIO2
- Q4 pad 2: Net-(Q3-D-Pad1) -> Net-(Q4-D)
- Q4 pad 3: Net-(Q4-G) -> GND
- R1 pad 1: +3V3 -> SCK
- R1 pad 2: /SCL_I2C -> Net-(J1-Pin_3)
- R10 pad 1: Net-(JP1-B) -> MOSI
- R10 pad 2: Net-(D2-A) -> Net-(U1-IO11)
- R11 pad 1: Net-(JP2-B) -> SCK
- R11 pad 2: Net-(D3-A) -> Net-(U1-IO12)
- R12 pad 1: Net-(JP3-A) -> Net-(C6-Pad2)
- R12 pad 2: /CS_GPS -> Net-(U1-IO15)
- R13 pad 1: Net-(C10-Pad1) -> Net-(C7-Pad2)
- R13 pad 2: /GNSS/VCC_RF -> Net-(U1-IO16)
- R14 pad 1: /MISO -> Net-(U1-USB_D-)
- R14 pad 2: Net-(U2-TXD/SPI_MISO) -> USB D-
- R15 pad 1: +3V3 -> Net-(U1-USB_D+)
- R15 pad 2: /NRST_LORA -> USB D+
- R16 pad 1: /MISO -> UART0_TX
- R16 pad 2: Net-(U3-MISO) -> Net-(J6-Pin_2)
- R17 pad 1: /EN_LORA -> UART0_RX
- R17 pad 2: GND -> Net-(J6-Pin_3)
- R18 pad 1: Net-(Q1-G) -> /Root/LoRa/EN
- R18 pad 2: -BATT -> /Root/GPIO_41
- R19 pad 1: Net-(U4-V-) -> /Root/GPIO_40
- R19 pad 2: GND -> /Root/LoRa/RESET
- R2 pad 1: +3V3 -> MOSI
- R2 pad 2: /SDA_I2C -> Net-(J1-Pin_4)
- R20 pad 1: +BATT -> Net-(JP3-B)
- R20 pad 2: Net-(U4-BAT) -> +3V3
- R21 pad 1: Net-(U3-DIO2) -> Net-(JP4-B)
- R21 pad 2: /TR_CTRL -> +3V3
- R22 pad 1: Net-(U7-PG) -> Net-(JP5-B)
- R22 pad 2: Net-(U7-VOUT) -> +3V3
- R23 pad 1: VBUS -> /Root/GPIO_10
- R23 pad 2: Net-(U6-PR1) -> +3V3
- R24 pad 1: GND -> /Root/CS_DISPLAY
- R24 pad 2: Net-(U6-PR1) -> +3V3
- R25 pad 1: +BATT -> /Root/CS_BUS
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Routing:
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- removed copper zone on In2.Cu, net +3V3
- removed copper zone on F.Cu, net Net-(U7-EN)
- removed copper zone on In1.Cu, net Net-(U7-EN)
- removed copper zone on F.Cu, net Net-(U7-VOUT)
- removed copper zone on In1.Cu, net Net-(U7-VOUT)
- removed copper zone on In1.Cu, net VBUS
- removed copper zone on In2.Cu, net VBUS
Other:
- board size 55 x 100 mm -> 60 x 130 mm
- board text removed: "+"
- board text removed: "-"
- board text removed: "18650 LITHIUM-ION ONLY"
- board text removed: "3V3"
- board text removed: "3V3 POWER"
- board text removed: ":3"
- board text removed: "BATTERY"
- board text removed: "CS_BUS"
- board text removed: "GND"
- board text removed: "GNSS"
- board text removed: "IPEX"
- board text removed: "John's Diner - Nightmaraze"
- board text removed: "LORA"
- board text removed: "LimesKey"
- board text removed: "MISO"
- board text removed: "MOSI"
- board text removed: "PPS (GNSS)"
- board text removed: "SCK"
- board text removed: "SCL_I2C"
- board text removed: "SDA_I2C"
- board text removed: "SMA LORA"
- board text removed: "SMA/IPEX"
- board text removed: "VBUS"
