File: parsnip.kicad_pcb (KiCad board)
At the start: 4 copper layers, 60 x 130 mm, 455 parts, among them J1 SPI BUS, J10 SOLAR, J11 Conn_Coaxial, J12 Conn_Coaxial_Small, J13 Conn_Coaxial, J14 GPIO_Expander, J15 LED 5V, J2 I2C3, J3 I2C1, J4 I2C2, J5 e-Ink Display Connector, J6 UART0, J7 GCT USB4105-GF-A-120, J8 PD_I2C DEBUG, J9 BAT_PORT, Q1 CSD25480F3, Q10 SI2308, Q11 CSD17581Q3A, Q12 AO3401A, Q13 BSS138, Q14 2N7002, Q15 2N7002, Q2 CSD15380F3, Q3 CSD25480F3, Q4 CSD15380F3, Q5 AON7534, Q6 AON7534, Q7 CSD18512Q5B, Q8 CSD18512Q5B, Q9 SI2308, SW1 ESP_RESET, SW2 BOOT, SW3 POWER/RESET, SW4 RESET_GNSS, SW5 SAFEBOOT_GNSS, U1 ESP32-S3-WROOM-1-N16R8, U10 TPS7A2033PDBVR, U11 TPS259474LRPWR, U12 E22P-915M30S, U13 LM61460AASQRJRRQ1, U14 LM61460AASQRJRRQ1, U15 TPS259474ARPWR, U16 SN74LVC1G74, U17 TCAL9539RTWR, U18 WS2816B, U19 SN74LV1T34DCK, U2 QMC6309, U20 WS2816B, U3 TVS2200DRV, U4 TPD8S300/A, U5 TI TPS25751DREFR, U6 CAT24C256, U7 MAX17320G22+, U8 BQ25798, U9 NEO-M9N, Y1 32.768KHz, Y2 SX1M4.000M10F30TNN

Commit message: add 3d models locally
Parts:
- D14: footprint Diode_SMD:D_0402_1005Metric -> Package_SON:Texas_DPY0002A_0.6x1mm_P0.65mm
- U6: footprint Package_DFN_QFN:OnSemi_UDFN-8_1.2x1.8mm_P0.4mm -> Package_DFN_QFN:DFN-8-1EP_2x3mm_P0.5mm_EP0.61x2.2mm
- moved C2 7.72 mm to (141.3, 137.9)
- moved F1 4.44 mm to (141.3, 135.4), turned to -90 degrees
