File: gnss.kicad_sch (KiCad schematic)
At the start: 72 parts, among them J11 Conn_Coaxial, J12 Conn_Coaxial_Small, Q12 AO3401A, Q13 BSS138, SW4 RESET_GNSS, SW5 SAFEBOOT_GNSS, U10 TPS7A2033PDBVR, U11 TPS259474LRPWR, U9 NEO-M9N

Commit message: done pcb layout
Parts:
- removed JP8, JP9: TIMEPULSE, Jumper:SolderJumper-2_P1.3mm_Bridged_RoundedPad1.0x1.5mm, symbol Jumper:SolderJumper_2_Bridged
- added C183: 1uF, Capacitor_SMD:C_0402_1005Metric, symbol Device:C_Small
- C100: value 100nF -> 1uF; LCSC Part C5272680 -> C53426846; Voltage Rating 50V -> 25V
- C103: value 1uF -> 10uF; LCSC Part C7472948 -> C6119763
- JP11: footprint Jumper:SolderJumper-3_P1.3mm_Open_RoundedPad1.0x1.5mm_NumberLabels -> Jumper:SolderJumper-3_P1.3mm_Bridged12_RoundedPad1.0x1.5mm
- R88: footprint Resistor_SMD:R_0603_1608Metric_Pad0.98x0.95mm_HandSolder -> Resistor_SMD:R_0402_1005Metric_Pad0.72x0.64mm_HandSolder; LCSC Part C47125286 -> (none)
Connections:
- net +3V3: no longer R91.1
- net 3V3_GNSS: now also R70.1, R91.1
- net GND: now also C183.2
- net PPS: now also R71.1
- net SCL/SPI_CLK: now also R72.2; no longer R68.2
- net SDA/SPI_CS: now also R68.2; no longer R72.2
- net VCC_RF: now also C183.1
Other:
- company: Ryan Di Lorenzo -> LimesKey
- moved on the sheet: JP10, R68, R70, R72, SW5
