File: gnss.kicad_sch (KiCad schematic)
At the start: 71 parts, among them J11 Conn_Coaxial, J12 Conn_Coaxial_Small, Q12 AO3401A, Q13 BSS138, SW4 RESET_GNSS, SW5 SAFEBOOT_GNSS, U10 TPS7A2033PDBVR, U11 TPS259474LRPWR, U9 NEO-M9N

Commit message: add 3d models locally
Parts:
- D14: footprint Diode_SMD:D_0402_1005Metric -> Package_SON:Texas_DPY0002A_0.6x1mm_P0.65mm
Changed lines of the file:
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@@
 			)
 		)
-		(property "Footprint" "Diode_SMD:D_0402_1005Metric"
+		(property "Footprint" "Package_SON:Texas_DPY0002A_0.6x1mm_P0.65mm"
 			(at 111.76 30.48 0)
 			(hide yes)

Commit message: progress in layout!
Parts:
- removed C107: 100nF, Capacitor_SMD:C_0402_1005Metric, symbol Device:C_Small
- removed C98: 10uF, Capacitor_SMD:C_0603_1608Metric, symbol Device:C_Small
- removed TP5: CS_GPS, TestPoint:TestPoint_Loop_D1.80mm_Drill1.0mm_Beaded, symbol Connector:TestPoint_Probe
- added TP5: CS_GPS, TestPoint:TestPoint_2Pads_Pitch2.54mm_Drill0.8mm, symbol Connector:TestPoint_2Pole
Connections:
- net GND: now also TP5.1
- net SDA/SPI_CS: now also TP5.2
Other:
- moved on the sheet: C106, D17
