File: peripherals.kicad_sch (KiCad schematic)
At the start: 13 parts, among them J14 GPIO_Expander, U17 TCAL9539RTWR, U18 WS2816B, U19 SN74LV1T34DCK, U2 QMC6309, U20 WS2816B

Commit message: done pcb layout
Parts:
- added C16: 10uF, Capacitor_SMD:C_0603_1608Metric, symbol Device:C_Small
- added F6: 3A hold 5A trip, Fuse:Fuse_1812_4532Metric, symbol Device:Polyfuse
- added J15: LED 5V, Connector_JST:JST_XH_S4B-XH-SM4-TB_1x04-1MP_P2.50mm_Horizontal, symbol Connector_Generic_MountingPin:Conn_01x04_MountingPin
- added R133: 10k, Resistor_SMD:R_0402_1005Metric_Pad0.72x0.64mm_HandSolder, symbol Device:R_Small
- J14: footprint Connector_PinSocket_2.54mm:PinSocket_2x08_P2.54mm_Horizontal -> easyeda2kicad:HDR-SMD_16P-P2.54_HXPM2.54-2X8PWT; LCSC Part C239359 -> C46635853
Connections:
- net +3V3: now also R133.2
- net +5V: now also C16.1, F6.1
- net GND: now also J14.14 (Pin_14), J14.16 (Pin_16), C16.2, J15.4 (Pin_4), J15.MP (MountPin)
- net RESET_IOEXP: now also R133.1
- net LED_BDO: now reaches U20.1 (BO)
- net LED_BDO: now also J15.3 (Pin_3)
- net LED_DO: now reaches U20.3 (DO)
- net LED_DO: now also J15.2 (Pin_2)
- net P16 renamed IO_P16
- net IO_P16: no longer J14.14 (Pin_14)
- net P17 renamed IO_P17
- net IO_P17: no longer J14.16 (Pin_16)
- new net: F6.2, J15.1 (Pin_1)
Other:
- note added: "For use with WS2813/WS2816"
- note added: "GPIO Expander"
- note added: "Individually Addressible RGB LEDs"
- company: (none) -> LimesKey
- title: (none) -> GPIO Expander / LEDs / Magnetometer
- moved on the sheet: C176, C177, C178, C179, C180, J14, U17, U18, U19, U20
