File: lora.kicad_sch (KiCad schematic)
At the start: 31 parts, among them J9 Conn_Coaxial, Q10 2N7002, U11 E22P-915M30S

Commit message: journal update!
Parts:
- added R123: 100k, Resistor_SMD:R_0402_1005Metric, symbol Device:R_Small
- C102: Capacitor Rating (none) -> X7R; LCSC Part (none) -> C5142567; Voltage Rating (none) -> 50V
Connections:
- net +3V3: now also R123.1
- net CS: now also R123.2

Commit message: pcb layout!
Parts:
- removed R81: 100, Resistor_SMD:R_0402_1005Metric, symbol Device:R_Small
- C112: renamed from C98; footprint (none) -> Capacitor_SMD:C_0402_1005Metric; LCSC Part (none) -> C54916656
- C113: renamed from C99; value 1pF C0G -> 1pF; Capacitor Rating (none) -> C0G
- C114: renamed from C100; value 1pF C0G -> 1pF; Capacitor Rating (none) -> C0G
- C115: renamed from C101; value 47pF C0G/NP0 -> 47pF; Capacitor Rating (none) -> C0G; LCSC Part (none) -> C20069324
- C116: renamed from C102; LCSC Part C5142567 -> C5272680
- C117: renamed from C103; LCSC Part (none) -> C7472948
- C118: renamed from C104; LCSC Part (none) -> C7472948
- C119: renamed from C105; footprint Capacitor_SMD:C_0805_2012Metric -> Capacitor_SMD:C_1206_3216Metric; LCSC Part (none) -> C12891
- C120: renamed from C106; footprint Capacitor_SMD:C_0805_2012Metric -> Capacitor_SMD:C_1206_3216Metric; LCSC Part (none) -> C12891
- C121: renamed from C107; footprint (none) -> Capacitor_SMD:C_0402_1005Metric; Capacitor Rating (none) -> X7R; LCSC Part (none) -> C5272680; Voltage Rating (none) -> 50V
- D18: renamed from D14; LCSC Part (none) -> C10677
- L3: footprint (none) -> Inductor_SMD:L_0603_1608Metric; LCSC Part (none) -> C113132
- Q14: renamed from Q10; LCSC Part (none) -> C5331134
- R100: renamed from R80; LCSC Part (none) -> C17477
- R101: renamed from R82; LCSC Part (none) -> C2902636
- R102: renamed from R83; footprint (none) -> Resistor_SMD:R_0402_1005Metric; LCSC Part (none) -> C2918201
- R92: renamed from R73; footprint (none) -> Resistor_SMD:R_0402_1005Metric; LCSC Part (none) -> C2902636
- R93: renamed from R74; LCSC Part (none) -> C844711
- R94: renamed from R75; LCSC Part (none) -> C2902636
- R95: renamed from R76; LCSC Part (none) -> C844711
- R96: renamed from R123; LCSC Part (none) -> C2984406
- R97: renamed from R77; LCSC Part (none) -> C2902636
- R98: renamed from R78; LCSC Part (none) -> C2686485
- R99: renamed from R79; footprint (none) -> Resistor_SMD:R_0402_1005Metric; LCSC Part (none) -> C48533754
- renumbered D15 to D19, J9 to J13, JP13 to JP14, JP14 to JP15, U11 to U12

Commit message: done pcb layout
Parts:
- removed TP6: 5V_LORA, TestPoint:TestPoint_2Pads_Pitch2.54mm_Drill0.8mm, symbol Connector:TestPoint_2Pole
Other:
- company: Ryan Di Lorenzo -> LimesKey
Changed lines of the file:
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@@
 		(title "LoRa Module / LoRa Antenna")
 		(date "2026-08-24")
-		(company "Ryan Di Lorenzo")
+		(company "LimesKey")
 	)
 	(rectangle
@@
 	)
 	(junction
-		(at 213.36 81.28)
-		(diameter 0)
-		(color 0 0 0 0)
-	)
-	(junction
 		(at 195.58 73.66)
 		(diameter 0)
@@
 	)
 	(junction
-		(at 195.58 86.36)
-		(diameter 0)
-		(color 0 0 0 0)
-	)
-	(junction
 		(at 195.58 83.82)
 		(diameter 0)
@@
 	(wire
 		(pts
-			(xy 213.36 81.28) (xy 213.36 86.36)
-		)
-		(stroke
-			(width 0)
-			(type default)
-		)
-	)
-	(wire
-		(pts
 			(xy 116.84 163.83) (xy 116.84 162.56)
 		)
@@
 	(wire
 		(pts
-			(xy 195.58 86.36) (xy 199.39 86.36)
-		)
-		(stroke
-			(width 0)
-			(type default)
-		)
-	)
-	(wire
-		(pts
 			(xy 104.14 170.18) (xy 90.17 170.18)
 		)
@@
 	(wire
 		(pts
-			(xy 153.67 104.14) (xy 156.21 104.14)
+			(xy 147.32 104.14) (xy 156.21 104.14)
 		)
 		(stroke
@@
 	(wire
 		(pts
-			(xy 209.55 86.36) (xy 213.36 86.36)
-		)
-		(stroke
-			(width 0)
-			(type default)
-		)
-	)
-	(wire
-		(pts
 			(xy 49.53 172.72) (xy 50.8 172.72)
 		)
@@
 	)
 	(label "LORA_ANT"
-		(at 153.67 104.14 180)
+		(at 147.32 104.14 180)
 		(effects
 			(font
@@
 		(dnp no)
 		(property "Reference" "R101"
-			(at 194.056 97.028 0)
+			(at 192.786 97.282 0)
 			(show_name no)
 			(do_not_autoplace no)
@@
 	)
 	(symbol
-		(lib_id "Connector:TestPoint_2Pole")
-		(at 204.47 86.36 0)
-		(unit 1)
-		(body_style 1)
-		(exclude_from_sim no)
-		(in_bom no)
-		(on_board yes)
-		(in_pos_files yes)
-		(dnp no)
-		(property "Reference" "TP6"
-			(at 204.47 88.138 0)
-			(show_name no)
-			(do_not_autoplace no)
-			(effects
-				(font
-					(size 1.27 1.27)
-				)
-			)
-		)
-		(property "Value" "5V_LORA"
-			(at 204.216 88.392 0)
-			(hide yes)
-			(show_name no)
-			(do_not_autoplace no)
-			(effects
-				(font
-					(size 1.27 1.27)
-				)
-			)
-		)
-		(property "Footprint" "TestPoint:TestPoint_2Pads_Pitch2.54mm_Drill0.8mm"
-			(at 204.47 86.36 0)
-			(hide yes)
-			(show_name no)
-			(do_not_autoplace no)
-			(effects
-				(font
-					(size 1.27 1.27)
-				)
-			)
-		)
-		(property "Datasheet" ""
-			(at 204.47 86.36 0)
-			(hide yes)
-			(show_name no)
-			(do_not_autoplace no)
-			(effects
-				(font
-					(size 1.27 1.27)
-				)
-			)
-		)
-		(property "Description" "2-polar test point"
-			(at 204.47 86.36 0)
-			(hide yes)
-			(show_name no)
-			(do_not_autoplace no)
-			(effects
-				(font
-					(size 1.27 1.27)
-				)
-			)
-		)
-		(property "LCSC Part" ""
-			(at 204.47 86.36 0)
-			(hide yes)
-			(show_name no)
-			(do_not_autoplace no)
-			(effects
-				(font
-					(size 1.27 1.27)
-				)
-			)
-		)
-		(property "Voltage Rating" ""
-			(at 204.47 86.36 0)
-			(hide yes)
-			(show_name no)
-			(do_not_autoplace no)
-			(effects
-				(font
-					(size 1.27 1.27)
-				)
-			)
-		)
-		(property "Tolerance" ""
-			(at 204.47 86.36 0)
-			(hide yes)
-			(show_name no)
-			(do_not_autoplace no)
-			(effects
-				(font
-					(size 1.27 1.27)
-				)
-			)
-		)
-		(pin "1"
-		)
-		(pin "2"
-		)
-		(instances
-			(project "parsnip"
-				(path "/fe9d4a31-2311-442f-997c-52ad8ca5cfe9/a8463f07-c31a-442f-966c-3f51ff19a9b1"
-					(reference "TP6")
-					(unit 1)
-				)
-			)
-		)
-	)
-	(symbol
 		(lib_id "Device:R_Small")
 		(at 195.58 64.77 0)
@@
 		)
 		(property "Value" "100nF"
-			(at 134.62 94.488 0)
+			(at 130.302 93.98 0)
 			(show_name no)
 			(do_not_autoplace no)

Commit message: slightly better component placement
Other:
- note added: "DC-shorted antenna only unless JP8 is cut Passive antenna only"
- note removed: "DC-shorted antenna only unless JP8 is cut"
Changed lines of the file:
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@@
 		)
 	)
-	(text "DC-shorted antenna only unless JP8 is cut"
+	(text "DC-shorted antenna only unless JP8 is cut\nPassive antenna only"
 		(exclude_from_sim no)
-		(at 75.184 139.446 0)
+		(at 80.518 138.938 0)
 		(effects
 			(font
