File: rails.kicad_sch (KiCad schematic)
At the start: 105 parts, among them Q15 2N7002, U13 LM61460AASQRJRRQ1, U14 LM61460AASQRJRRQ1, U15 TPS259474ARPWR, U16 SN74LVC1G74, Y2 SX1M4.000M10F30TNN

Commit message: done pcb layout
Parts:
- added TP16: SYNC_3V3, TestPoint:TestPoint_Pad_D1.0mm, symbol Connector:TestPoint_Probe
- added TP6: SYNC_5V, TestPoint:TestPoint_Pad_D1.0mm, symbol Connector:TestPoint_Probe
- C132, C138: footprint Capacitor_SMD:C_0402_1005Metric -> Capacitor_SMD:C_0603_1608Metric; LCSC Part C53426846 -> C7432774; Voltage Rating 25V -> 50V
Connections:
- net GND: now also C132.1, C138.1; no longer C132.2, C138.2
- net SYNC_1: now also TP6.1
- net SYNC_2: now also TP16.1
- net VSYS: now also C132.2, C138.2; no longer C132.1, C138.1
Other:
- note added: "2 x 10uF 1206"
- note removed: "2 x 10uF 1210"
- company: Ryan Di Lorenzo -> LimesKey

Commit message: progress in layout!
Parts:
- removed C140: 1uF, Capacitor_SMD:C_0402_1005Metric, symbol Device:C_Small
- removed C142, C152: 10uF, Capacitor_SMD:C_0603_1608Metric, symbol Device:C_Small
- removed C170, C171: 22uF, Capacitor_SMD:C_1206_3216Metric, symbol Device:C_Small
- removed TP16: SYNC_3V3, TestPoint:TestPoint_Pad_D1.0mm, symbol Connector:TestPoint_Probe
- removed TP6: SYNC_5V, TestPoint:TestPoint_Pad_D1.0mm, symbol Connector:TestPoint_Probe
- added C185, C186, C187: 22uF, Capacitor_SMD:C_1206_3216Metric, symbol Device:C_Small
- added TP16: SYNC_2, TestPoint:TestPoint_2Pads_Pitch2.54mm_Drill0.8mm, symbol Connector:TestPoint_2Pole
- added TP6: SYNC_1, TestPoint:TestPoint_2Pads_Pitch2.54mm_Drill0.8mm, symbol Connector:TestPoint_2Pole
- C147: value 1uF -> 22uF; footprint Capacitor_SMD:C_0402_1005Metric -> Capacitor_SMD:C_1206_3216Metric; LCSC Part C53426846 -> C48579675
- C157: value 1uF -> 22uF; footprint Capacitor_SMD:C_0402_1005Metric -> Capacitor_SMD:C_1206_3216Metric; LCSC Part C53426846 -> C48579675; Voltage Rating 25V -> 16V
- C169: value 22uF -> 10uF; footprint Capacitor_SMD:C_1206_3216Metric -> Capacitor_SMD:C_0603_1608Metric; LCSC Part C48579675 -> C22392391
- TP10, TP11: footprint TestPoint:TestPoint_Loop_D2.54mm_Drill1.5mm_Beaded -> TestPoint:TestPoint_Pad_D1.5mm
- TP7: footprint TestPoint:TestPoint_Pad_D1.5mm -> TestPoint:TestPoint_Pad_D1.0mm
Connections:
- net +3V3: now also C147.1, C185.1
- net 5V_RAW: now also C157.1, C186.1, C187.2; no longer C147.1, C157.2
- net GND: now also C157.2, C185.2, C186.2, C187.1, TP16.1, TP6.1; no longer C157.1
- net SYNC_1: now also TP6.2
- net SYNC_2: now also TP16.2
Other:
- moved on the sheet: C156, C159, C160, C163, C164, C167, C168, C174, D21, D22, R132, U16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
